Commit message: New launches and robots for trials

File: softfoot_thing_description/robot/vertical_softfoot.urdf.xacro (robot description, xacro)
@@ -9,6 +9,9 @@
 </link>
 <!-- LEG -->
-<joint name="world_to_leg" type="floating">
+<joint name="world_to_leg" type="prismatic">
     <origin xyz="0 0 0.5" rpy="0 0 0"/>
+    <axis xyz="0 0 -1"/>
+    <limit lower="-0.50" upper="0.50" effort="1" velocity="1" />
+    <dynamics friction="0.0" damping="0.0"/>
     <parent link="world"/>
     <child link="leg_link"/>
