Commit message: Added robot

File: softfoot_thing_description/robot/pisa_softfoot.urdf.xacro (robot description, xacro)
@@ -1,14 +1,12 @@
 <?xml version="1.0" encoding='utf-8'?>
-<robot xmlns:xacro="http://www.ros.org/wiki/xacro" name="softfoot_thing">
+<robot xmlns:xacro="http://www.ros.org/wiki/xacro" name="pisa_softfoot">
   <!-- ARGS -->
   <!-- MODELS -->
+  <xacro:include filename="$(find softfoot_thing_description)/model/softfoot_thing.urdf.xacro"/>
   <!-- WORLD -->
-  <!-- <link name="world"/>
-  <joint name="world_to_foot" type="fixed">
+  <link name="world"/>
+  <!-- FOOT -->
+  <xacro:softfoot_thing name="pisa_softfoot" parent="world">
     <origin xyz="0 0 0" rpy="0 0 0"/>
-    <parent link="world" />
-    <child link="foot_link0" />
-  </joint> -->
-  <!-- FOOT -->
-  <!-- <xacro:softfoot_thing /> -->
+  </xacro:softfoot_thing>
 </robot>

Commit message: Typo

File: softfoot_thing_description/robot/pisa_softfoot.urdf.xacro (robot description, xacro)
@@ -8,5 +8,5 @@
   <!-- LEG -->
   <joint name="world_to_leg" type="fixed">
-    <origin xyz="0 0 0.2" rpy="0 0 0"/>
+    <origin xyz="0 0 0.2" rpy="0.0 0.0 0.0"/>
     <parent link="world"/>
     <child link="leg_link"/>

Commit message: orientation change

File: softfoot_thing_description/robot/pisa_softfoot.urdf.xacro (robot description, xacro)
@@ -8,5 +8,5 @@
   <!-- LEG -->
   <joint name="world_to_leg" type="fixed">
-    <origin xyz="0 0 0.2" rpy="0.57 0.57 0.57"/>
+    <origin xyz="0 0 0.2" rpy="0.0 0.0 0.0"/>
     <parent link="world"/>
     <child link="leg_link"/>

Commit message: Added inertial to leg link

File: softfoot_thing_description/robot/pisa_softfoot.urdf.xacro (robot description, xacro)
@@ -2,8 +2,13 @@
 <robot xmlns:xacro="http://www.ros.org/wiki/xacro" name="pisa_softfoot">
   <!-- ARGS -->
+  <xacro:property name="leg_mass" value="0.02"/>
   <!-- MODELS -->
   <xacro:include filename="$(find softfoot_thing_description)/model/softfoot_thing.urdf.xacro"/>
   <!-- WORLD -->
-  <link name="world"/>
+  <link name="world">
+    <inertial>
+      <xacro:insert_block name="negligible_inertia"/>
+    </inertial>
+  </link>
   <!-- LEG -->
   <joint name="world_to_leg" type="fixed">
@@ -13,12 +18,23 @@
   </joint>
   <link name="leg_link">
+    <inertial>
+			<mass value="${leg_mass}"/>
+			<origin xyz="0 0 0" rpy="0 0 0"/>
+			<inertia  ixx="${mm2tom2 * 1}" iyy="${mm2tom2 * 1}" izz="${mm2tom2 * 1}"
+                ixy="0" ixz="0" iyz="0"/>
+		</inertial>
     <visual>
+      <origin xyz="0 0 0" rpy="0 0 0"/>
       <geometry>
         <cylinder length="0.1" radius="0.015"/>
       </geometry>
-      <material name="material.metal">
-        <color rgba="0.1 0.1 0.1 1" />
-      </material>
+      <material name="SoftFoot/Black"/>
     </visual>
+    <collision>
+			<origin xyz="0 0 0" rpy="0 0 0"/>
+			<geometry>
+        <cylinder length="0.1" radius="0.015"/>
+      </geometry>
+		</collision>
   </link>
   <!-- FOOT -->

Commit message: No need for inertia in root link

File: softfoot_thing_description/robot/pisa_softfoot.urdf.xacro (robot description, xacro)
@@ -7,11 +7,8 @@
   <!-- WORLD -->
   <link name="world">
-    <inertial>
-      <xacro:insert_block name="negligible_inertia"/>
-    </inertial>
   </link>
   <!-- LEG -->
   <joint name="world_to_leg" type="fixed">
-    <origin xyz="0 0 0.2" rpy="0.78 0.78 0.78"/>
+    <origin xyz="0 0 0.2" rpy="0 0 0"/>
     <parent link="world"/>
     <child link="leg_link"/>

Commit message: Added softfoot 4

File: softfoot_thing_description/robot/pisa_softfoot.urdf.xacro (robot description, xacro)
@@ -8,11 +8,11 @@
   <link name="world">
   </link>
-  <!-- LEG -->
-  <joint name="world_to_leg" type="fixed">
+  <!-- LEG 1 -->
+  <joint name="world_to_leg_1" type="fixed">
     <origin xyz="0 0 0.2" rpy="0 0 0"/>
     <parent link="world"/>
-    <child link="leg_link"/>
+    <child link="leg_link_1"/>
   </joint>
-  <link name="leg_link">
+  <link name="leg_link_1">
     <inertial>
 			<mass value="${leg_mass}"/>
@@ -35,10 +35,45 @@
 		</collision>
   </link>
-  <gazebo reference="leg_link">
+  <gazebo reference="leg_link_1">
 			<gravity>true</gravity>
 			<material>Gazebo/Black</material>
 		</gazebo>
-  <!-- FOOT -->
-  <xacro:softfoot_thing name="softfoot_3" parent="leg_link">
+  <!-- FOOT 1 -->
+  <xacro:softfoot_thing name="softfoot_3" parent="leg_link_1">
+    <origin xyz="0 0 -0.05" rpy="0 0 0"/>
+  </xacro:softfoot_thing>
+  <!-- LEG 2 -->
+  <joint name="world_to_leg_2" type="fixed">
+    <origin xyz="0 0.2 0.2" rpy="0 0 0"/>
+    <parent link="world"/>
+    <child link="leg_link_2"/>
+  </joint>
+  <link name="leg_link_2">
+    <inertial>
+			<mass value="${leg_mass}"/>
+			<origin xyz="0 0 0" rpy="0 0 0"/>
+			<inertia  ixx="${mm2tom2 * 1}" iyy="${mm2tom2 * 1}" izz="${mm2tom2 * 1}"
+                ixy="0" ixz="0" iyz="0"/>
+		</inertial>
+    <visual>
+      <origin xyz="0 0 0" rpy="0 0 0"/>
+      <geometry>
+        <cylinder length="0.1" radius="0.015"/>
+      </geometry>
+      <material name="SoftFoot/Black"/>
+    </visual>
+    <collision>
+			<origin xyz="0 0 0" rpy="0 0 0"/>
+			<geometry>
+        <cylinder length="0.1" radius="0.015"/>
+      </geometry>
+		</collision>
+  </link>
+  <gazebo reference="leg_link_2">
+			<gravity>true</gravity>
+			<material>Gazebo/Black</material>
+		</gazebo>
+  <!-- FOOT 2 -->
+  <xacro:softfoot_thing name="softfoot_4" parent="leg_link_2">
     <origin xyz="0 0 -0.05" rpy="0 0 0"/>
   </xacro:softfoot_thing>

Commit message: Removed one foot in master branch

File: softfoot_thing_description/robot/pisa_softfoot.urdf.xacro (robot description, xacro)
@@ -36,7 +36,7 @@
   </link>
   <gazebo reference="leg_link_1">
-			<gravity>true</gravity>
-			<material>Gazebo/Black</material>
-		</gazebo>
+		<gravity>true</gravity>
+		<material>Gazebo/Black</material>
+	</gazebo>
   <!-- FOOT 1 -->
   <xacro:softfoot_thing name="softfoot_3" parent="leg_link_1">
@@ -44,5 +44,5 @@
   </xacro:softfoot_thing>
   <!-- LEG 2 -->
-  <joint name="world_to_leg_2" type="fixed">
+  <!-- <joint name="world_to_leg_2" type="fixed">
     <origin xyz="0 0.2 0.2" rpy="0 0 0"/>
     <parent link="world"/>
@@ -73,8 +73,8 @@
 			<gravity>true</gravity>
 			<material>Gazebo/Black</material>
-		</gazebo>
+		</gazebo> -->
   <!-- FOOT 2 -->
-  <xacro:softfoot_thing name="softfoot_1" parent="leg_link_2">
+  <!-- <xacro:softfoot_thing name="softfoot_1" parent="leg_link_2">
     <origin xyz="0 0 -0.05" rpy="0 0 0"/>
-  </xacro:softfoot_thing>
+  </xacro:softfoot_thing> -->
 </robot>

Commit message: Trying two feet. IMUs should be of same orientation on all feet.

File: softfoot_thing_description/robot/pisa_softfoot.urdf.xacro (robot description, xacro)
@@ -44,5 +44,5 @@
   </xacro:softfoot_thing>
   <!-- LEG 2 -->
-  <!-- <joint name="world_to_leg_2" type="fixed">
+  <joint name="world_to_leg_2" type="fixed">
     <origin xyz="0 0.2 0.2" rpy="0 0 0"/>
     <parent link="world"/>
@@ -71,10 +71,10 @@
   </link>
   <gazebo reference="leg_link_2">
-			<gravity>true</gravity>
-			<material>Gazebo/Black</material>
-		</gazebo> -->
+		<gravity>true</gravity>
+		<material>Gazebo/Black</material>
+	</gazebo>
   <!-- FOOT 2 -->
-  <!-- <xacro:softfoot_thing name="softfoot_1" parent="leg_link_2">
+  <xacro:softfoot_thing name="softfoot_4" parent="leg_link_2">
     <origin xyz="0 0 -0.05" rpy="0 0 0"/>
-  </xacro:softfoot_thing> -->
+  </xacro:softfoot_thing>
 </robot>

Commit message: Got back to just foot 3

File: softfoot_thing_description/robot/pisa_softfoot.urdf.xacro (robot description, xacro)
@@ -44,5 +44,5 @@
   </xacro:softfoot_thing>
   <!-- LEG 2 -->
-  <joint name="world_to_leg_2" type="fixed">
+  <!-- <joint name="world_to_leg_2" type="fixed">
     <origin xyz="0 0.2 0.2" rpy="0 0 0"/>
     <parent link="world"/>
@@ -73,8 +73,8 @@
 		<gravity>true</gravity>
 		<material>Gazebo/Black</material>
-	</gazebo>
+	</gazebo> -->
   <!-- FOOT 2 -->
-  <xacro:softfoot_thing name="softfoot_4" parent="leg_link_2">
+  <!-- <xacro:softfoot_thing name="softfoot_4" parent="leg_link_2">
     <origin xyz="0 0 -0.05" rpy="0 0 0"/>
-  </xacro:softfoot_thing>
+  </xacro:softfoot_thing> -->
 </robot>

Commit message: Starting to write code to estimate leg pose aswell if requested

File: softfoot_thing_description/robot/pisa_softfoot.urdf.xacro (robot description, xacro)
@@ -9,10 +9,13 @@
   </link>
   <!-- LEG 1 -->
-  <joint name="world_to_leg_1" type="fixed">
+  <joint name="world_to_leg_3" type="revolute">
     <origin xyz="0 0 0.2" rpy="0 0 0"/>
+    <axis xyz="0 1 0"/>
+    <limit lower="-0.50" upper="0.50" effort="1" velocity="1" />
+		<dynamics friction="0.01" damping="0.01"/>
     <parent link="world"/>
-    <child link="leg_link_1"/>
+    <child link="leg_link_3"/>
   </joint>
-  <link name="leg_link_1">
+  <link name="leg_link_3">
     <inertial>
 			<mass value="${leg_mass}"/>
@@ -35,19 +38,19 @@
 		</collision>
   </link>
-  <gazebo reference="leg_link_1">
+  <gazebo reference="leg_link_3">
 		<gravity>true</gravity>
 		<material>Gazebo/Black</material>
 	</gazebo>
   <!-- FOOT 1 -->
-  <xacro:softfoot_thing name="softfoot_3" parent="leg_link_1">
+  <xacro:softfoot_thing name="softfoot_3" parent="leg_link_3">
     <origin xyz="0 0 -0.05" rpy="0 0 0"/>
   </xacro:softfoot_thing>
   <!-- LEG 2 -->
-  <!-- <joint name="world_to_leg_2" type="fixed">
+  <!-- <joint name="world_to_leg_4" type="fixed">
     <origin xyz="0 0.2 0.2" rpy="0 0 0"/>
     <parent link="world"/>
-    <child link="leg_link_2"/>
+    <child link="leg_link_4"/>
   </joint>
-  <link name="leg_link_2">
+  <link name="leg_link_4">
     <inertial>
 			<mass value="${leg_mass}"/>
@@ -70,10 +73,10 @@
 		</collision>
   </link>
-  <gazebo reference="leg_link_2">
+  <gazebo reference="leg_link_4">
 		<gravity>true</gravity>
 		<material>Gazebo/Black</material>
 	</gazebo> -->
   <!-- FOOT 2 -->
-  <!-- <xacro:softfoot_thing name="softfoot_4" parent="leg_link_2">
+  <!-- <xacro:softfoot_thing name="softfoot_4" parent="leg_link_4">
     <origin xyz="0 0 -0.05" rpy="0 0 0"/>
   </xacro:softfoot_thing> -->

Commit message: More realistic damping

File: softfoot_thing_description/robot/pisa_softfoot.urdf.xacro (robot description, xacro)
@@ -13,5 +13,5 @@
     <axis xyz="0 1 0"/>
     <limit lower="-0.50" upper="0.50" effort="1" velocity="1" />
-    <dynamics friction="0.01" damping="0.01"/>
+    <dynamics friction="0.0001" damping="0.0001"/>
     <parent link="world"/>
     <child link="leg_link_3"/>

Commit message: Modifications for new qb node

File: softfoot_thing_description/robot/pisa_softfoot.urdf.xacro (robot description, xacro)
@@ -9,5 +9,5 @@
 </link>
 <!-- LEG 1 -->
-<joint name="world_to_leg_3" type="revolute">
+<joint name="world_to_leg_1" type="revolute">
     <origin xyz="0 0 0.2" rpy="0 0 0"/>
     <axis xyz="0 1 0"/>
@@ -15,7 +15,7 @@
     <dynamics friction="0.0001" damping="0.0001"/>
     <parent link="world"/>
-    <child link="leg_link_3"/>
+    <child link="leg_link_1"/>
 </joint>
-<link name="leg_link_3">
+<link name="leg_link_1">
     <inertial>
         <mass value="${leg_mass}"/>
@@ -38,19 +38,22 @@
     </collision>
 </link>
-<gazebo reference="leg_link_3">
+<gazebo reference="leg_link_1">
     <gravity>true</gravity>
     <material>Gazebo/Black</material>
 </gazebo>
 <!-- FOOT 1 -->
-<xacro:softfoot_thing name="softfoot_3" parent="leg_link_3">
+<xacro:softfoot_thing name="softfoot_1" parent="leg_link_1">
     <origin xyz="0 0 -0.05" rpy="0 0 0"/>
 </xacro:softfoot_thing>
   <!-- LEG 2 -->
-  <!-- <joint name="world_to_leg_4" type="fixed">
-    <origin xyz="0 0.2 0.2" rpy="0 0 0"/>
-    <parent link="world"/>
-    <child link="leg_link_4"/>
-  </joint>
-  <link name="leg_link_4">
+    <joint name="world_to_leg_2" type="revolute">
+        <origin xyz="0 0.2 0.2" rpy="0 0 0"/>
+        <axis xyz="0 1 0"/>
+        <limit lower="-0.50" upper="0.50" effort="1" velocity="1" />
+        <dynamics friction="0.0001" damping="0.0001"/>
+        <parent link="world"/>
+        <child link="leg_link_2"/>
+    </joint>
+  <link name="leg_link_2">
     <inertial>
 			<mass value="${leg_mass}"/>
@@ -73,11 +76,87 @@
 		</collision>
   </link>
-  <gazebo reference="leg_link_4">
+  <gazebo reference="leg_link_2">
 		<gravity>true</gravity>
 		<material>Gazebo/Black</material>
-	</gazebo> -->
+	</gazebo>
   <!-- FOOT 2 -->
-  <!-- <xacro:softfoot_thing name="softfoot_4" parent="leg_link_4">
+ <xacro:softfoot_thing name="softfoot_2" parent="leg_link_2">
     <origin xyz="0 0 -0.05" rpy="0 0 0"/>
-  </xacro:softfoot_thing> -->
+  </xacro:softfoot_thing>
+    <!-- LEG 3 -->
+    <joint name="world_to_leg_3" type="revolute">
+        <origin xyz="0.2 0.2 0.2" rpy="0 0 0"/>
+        <axis xyz="0 1 0"/>
+        <limit lower="-0.50" upper="0.50" effort="1" velocity="1" />
+        <dynamics friction="0.0001" damping="0.0001"/>
+        <parent link="world"/>
+        <child link="leg_link_3"/>
+    </joint>
+    <link name="leg_link_3">
+        <inertial>
+            <mass value="${leg_mass}"/>
+            <origin xyz="0 0 0" rpy="0 0 0"/>
+            <inertia  ixx="${mm2tom2 * 1}" iyy="${mm2tom2 * 1}" izz="${mm2tom2 * 1}"
+                      ixy="0" ixz="0" iyz="0"/>
+        </inertial>
+        <visual>
+            <origin xyz="0 0 0" rpy="0 0 0"/>
+            <geometry>
+                <cylinder length="0.1" radius="0.015"/>
+            </geometry>
+            <material name="SoftFoot/Black"/>
+        </visual>
+        <collision>
+            <origin xyz="0 0 0" rpy="0 0 0"/>
+            <geometry>
+                <cylinder length="0.1" radius="0.015"/>
+            </geometry>
+        </collision>
+    </link>
+    <gazebo reference="leg_link_3">
+        <gravity>true</gravity>
+        <material>Gazebo/Black</material>
+    </gazebo>
+    <!-- FOOT 3 -->
+    <xacro:softfoot_thing name="softfoot_3" parent="leg_link_3">
+        <origin xyz="0 0 -0.05" rpy="0 0 0"/>
+    </xacro:softfoot_thing>
+    <!-- LEG 4 -->
+    <joint name="world_to_leg_4" type="revolute">
+        <origin xyz="0.2 0.0 0.2" rpy="0 0 0"/>
+        <axis xyz="0 1 0"/>
+        <limit lower="-0.50" upper="0.50" effort="1" velocity="1" />
+        <dynamics friction="0.0001" damping="0.0001"/>
+        <parent link="world"/>
+        <child link="leg_link_4"/>
+    </joint>
+    <link name="leg_link_4">
+        <inertial>
+            <mass value="${leg_mass}"/>
+            <origin xyz="0 0 0" rpy="0 0 0"/>
+            <inertia  ixx="${mm2tom2 * 1}" iyy="${mm2tom2 * 1}" izz="${mm2tom2 * 1}"
+                      ixy="0" ixz="0" iyz="0"/>
+        </inertial>
+        <visual>
+            <origin xyz="0 0 0" rpy="0 0 0"/>
+            <geometry>
+                <cylinder length="0.1" radius="0.015"/>
+            </geometry>
+            <material name="SoftFoot/Black"/>
+        </visual>
+        <collision>
+            <origin xyz="0 0 0" rpy="0 0 0"/>
+            <geometry>
+                <cylinder length="0.1" radius="0.015"/>
+            </geometry>
+        </collision>
+    </link>
+    <gazebo reference="leg_link_4">
+        <gravity>true</gravity>
+        <material>Gazebo/Black</material>
+    </gazebo>
+    <!-- FOOT 3 -->
+    <xacro:softfoot_thing name="softfoot_4" parent="leg_link_4">
+        <origin xyz="0 0 -0.05" rpy="0 0 0"/>
+    </xacro:softfoot_thing>
 </robot>

Commit message: Updated disposition of feet

File: softfoot_thing_description/robot/pisa_softfoot.urdf.xacro (robot description, xacro)
@@ -86,5 +86,5 @@
     <!-- LEG 3 -->
     <joint name="world_to_leg_3" type="revolute">
-        <origin xyz="0.2 0.2 0.2" rpy="0 0 0"/>
+        <origin xyz="-0.2 0.2 0.2" rpy="0 0 0"/>
         <axis xyz="0 1 0"/>
         <limit lower="-0.50" upper="0.50" effort="1" velocity="1" />
@@ -124,5 +124,5 @@
     <!-- LEG 4 -->
     <joint name="world_to_leg_4" type="revolute">
-        <origin xyz="0.2 0.0 0.2" rpy="0 0 0"/>
+        <origin xyz="-0.2 0.0 0.2" rpy="0 0 0"/>
         <axis xyz="0 1 0"/>
         <limit lower="-0.50" upper="0.50" effort="1" velocity="1" />

Commit message: Corrected configs

File: softfoot_thing_description/robot/pisa_softfoot.urdf.xacro (robot description, xacro)
@@ -10,5 +10,5 @@
 <!-- LEG 1 -->
 <joint name="world_to_leg_1" type="revolute">
-    <origin xyz="0 0 0.2" rpy="0 0 0"/>
+    <origin xyz="0 0.2  0.2" rpy="0 0 0"/>
     <axis xyz="0 1 0"/>
     <limit lower="-0.50" upper="0.50" effort="1" velocity="1" />
@@ -48,5 +48,5 @@
   <!-- LEG 2 -->
     <joint name="world_to_leg_2" type="revolute">
-        <origin xyz="0 0.2 0.2" rpy="0 0 0"/>
+        <origin xyz="0 0.0 0.2" rpy="0 0 0"/>
         <axis xyz="0 1 0"/>
         <limit lower="-0.50" upper="0.50" effort="1" velocity="1" />
