Commit message: Added prismatic joint in leg to approx. simulate walk

File: softfoot_thing_description/robot/floating_softfoot.urdf.xacro (robot description, xacro)
@@ -5,5 +5,16 @@
 <!-- MODELS -->
 <xacro:include filename="$(find softfoot_thing_description)/model/softfoot_thing.urdf.xacro"/>
-<!-- LEG 1 -->
+<!-- WORLD -->
+<link name="world">
+</link>
+<!-- LEG -->
+<joint name="world_to_leg" type="prismatic">
+    <origin xyz="0 0 0.5" rpy="0 0 0"/>
+    <axis xyz="0 0 -1"/>
+    <limit lower="-0.50" upper="0.50" effort="1" velocity="1" />
+    <dynamics friction="0.0" damping="0.0"/>
+    <parent link="world"/>
+    <child link="leg_link"/>
+</joint>
 <link name="leg_link">
     <inertial>

Commit message: Modified height

File: softfoot_thing_description/robot/floating_softfoot.urdf.xacro (robot description, xacro)
@@ -10,5 +10,5 @@
 <!-- LEG -->
 <joint name="world_to_leg" type="floating">
-    <origin xyz="0 0 0.5" rpy="0 0 0"/>
+    <origin xyz="0 0 0.17" rpy="0 0 0"/>
     <parent link="world"/>
     <child link="leg_link"/>
