Commit message: Corrected names and added inertial elements

File: softfoot_thing_description/model/softfoot_thing.urdf.xacro (robot description, xacro)
@@ -3,7 +3,7 @@
 	<!-- Properties -->
     <xacro:property name="const_pi" value="3.1415926535897931"/>
-	<xacro:property name="ankle_mass" value="0.1814"/>
-    <xacro:property name="harch_mass" value="2.35"/>
-    <xacro:property name="roll_mass" value="1.1"/>
+	<xacro:property name="ankle_mass" value="0.0181"/>
+    <xacro:property name="arch_mass" value="0.0256"/>
+    <xacro:property name="roll_mass" value="0.0177"/>
 	<xacro:property name="velocity_scale" value="1"/>
 	<xacro:property name="effort_scale" value="1"/>
@@ -27,6 +27,6 @@
 			<inertial>
 				<mass value="${ankle_mass}"/>
-				<origin xyz="0 0 0" rpy="0 0 0"/>
-				<cylinder_inertia_def radius="0.06" length="0.11" mass="${ankle_mass}"/>
+				<origin xyz="0 0 0.0154" rpy="0 0 0"/>
+				<ankle_inertia/>
 			</inertial>
 			<visual>
@@ -44,6 +44,6 @@
 			</collision>
 		</link>
-		<!-- 2) Front harch - joint along y-axis to pitch -->
-		<joint name="${name}_front_harch_joint" type="revolute">
+		<!-- 2) Front arch - joint along y-axis to pitch -->
+		<joint name="${name}_front_arch_joint" type="revolute">
 			<origin xyz="0 0 0" rpy="0 0 0"/>
 			<axis xyz="0 1 0"/>
@@ -51,16 +51,16 @@
 			<dynamics friction="10.0" damping="1.0"/>
 			<parent link="${name}_ankle_link"/>
-			<child link="${name}_front_harch_link"/>
-		</joint>
-		<link name="${name}_front_harch_link">
-			<inertial>
-				<mass value="${harch_mass}"/>
-				<origin xyz="0 -0.06 0.130" rpy="0 0 0"/>
-				<cuboid_inertia_def length="0.12" width="0.06" height="0.260" mass="${harch_mass}"/>
-			</inertial>
-			<visual>
-				<origin xyz="0 0 0" rpy="0 0 0"/>
-				<geometry>
-					<mesh filename="package://softfoot_thing_description/meshes/visual/front_harch_front.stl" scale=" .001 .001 .001"/>
+			<child link="${name}_front_arch_link"/>
+		</joint>
+		<link name="${name}_front_arch_link">
+			<inertial>
+				<mass value="${arch_mass}"/>
+				<origin xyz="0.0356 -0.0011 -0.0078" rpy="0 0 0"/>
+				<front_arch_inertia/>
+			</inertial>
+			<visual>
+				<origin xyz="0 0 0" rpy="0 0 0"/>
+				<geometry>
+					<mesh filename="package://softfoot_thing_description/meshes/visual/front_arch_front.stl" scale=" .001 .001 .001"/>
 				</geometry>
 				<material name="SoftFoot/Silver"/>
@@ -73,6 +73,6 @@
 			</collision>
 		</link>
-        <!-- 2) Front harch - stiffness -->
-        <joint name="${name}_front_harch_joint_stiffness" type="revolute">
+        <!-- 2) Front arch - stiffness -->
+        <joint name="${name}_front_arch_joint_stiffness" type="revolute">
             <origin xyz="0 0 0" rpy="0 0 0"/>
 			<axis xyz="0 1 0"/>
@@ -80,9 +80,9 @@
 			<safety_controller soft_lower_limit="${min_stiffness}" soft_upper_limit="${max_stiffness}" k_position="30" k_velocity="30"/>
 			<parent link="${name}_ankle_link"/>
-			<child link="${name}_front_harch_dummy"/>
-		</joint>
-		<link name="${name}_front_harch_dummy"/>
-        <!-- 3) Back harch - joint along y-axis to pitch -->
-		<joint name="${name}_back_harch_joint" type="revolute">
+			<child link="${name}_front_arch_dummy"/>
+		</joint>
+		<link name="${name}_front_arch_dummy"/>
+        <!-- 3) Back arch - joint along y-axis to pitch -->
+		<joint name="${name}_back_arch_joint" type="revolute">
 			<origin xyz="0 0 0" rpy="0 0 0"/>
 			<axis xyz="0 -1 0"/>
@@ -90,28 +90,28 @@
 			<dynamics friction="10.0" damping="1.0"/>
 			<parent link="${name}_ankle_link"/>
-			<child link="${name}_back_harch_link"/>
-		</joint>
-		<link name="${name}_back_harch_link">
-			<inertial>
-				<mass value="${harch_mass}"/>
-				<origin xyz="0 -0.06 0.130" rpy="0 0 0"/>
-				<cuboid_inertia_def length="0.12" width="0.06" height="0.260" mass="${harch_mass}"/>
-			</inertial>
-			<visual>
-				<origin xyz="0 0 0" rpy="0 0 0"/>
-				<geometry>
-					<mesh filename="package://softfoot_thing_description/meshes/visual/front_harch_back.stl" scale=" .001 .001 .001"/>
-				</geometry>
-				<material name="SoftFoot/Silver"/>
-			</visual>
-			<collision>
-				<origin xyz="0 0 0" rpy="0 0 0"/>
-				<geometry>
-					<sphere radius="0.07"/>
-				</geometry>
-			</collision>
-		</link>
-        <!-- 3) Back harch - stiffness -->
-        <joint name="${name}_back_harch_joint_stiffness" type="revolute">
+			<child link="${name}_back_arch_link"/>
+		</joint>
+		<link name="${name}_back_arch_link">
+			<inertial>
+				<mass value="${arch_mass}"/>
+				<origin xyz="-0.0356 0.0011 -0.0078" rpy="0 0 0"/>
+				<back_arch_inertia/>
+			</inertial>
+			<visual>
+				<origin xyz="0 0 0" rpy="0 0 0"/>
+				<geometry>
+					<mesh filename="package://softfoot_thing_description/meshes/visual/front_arch_back.stl" scale=" .001 .001 .001"/>
+				</geometry>
+				<material name="SoftFoot/Silver"/>
+			</visual>
+			<collision>
+				<origin xyz="0 0 0" rpy="0 0 0"/>
+				<geometry>
+					<sphere radius="0.07"/>
+				</geometry>
+			</collision>
+		</link>
+        <!-- 3) Back arch - stiffness -->
+        <joint name="${name}_back_arch_joint_stiffness" type="revolute">
             <origin xyz="0 0 0" rpy="0 0 0"/>
 			<axis xyz="0 -1 0"/>
@@ -119,7 +119,7 @@
 			<safety_controller soft_lower_limit="${min_stiffness}" soft_upper_limit="${max_stiffness}" k_position="30" k_velocity="30"/>
 			<parent link="${name}_ankle_link"/>
-			<child link="${name}_back_harch_dummy"/>
-		</joint>
-		<link name="${name}_back_harch_dummy"/>
+			<child link="${name}_back_arch_dummy"/>
+		</joint>
+		<link name="${name}_back_arch_dummy"/>
         <!-- x) Roll driving joint - we suppose the roll joints move specularly -->
 		<joint name="${name}_roll_joint" type="revolute">
@@ -128,5 +128,5 @@
 			<limit lower="${-45 * const_pi / 180}" upper="${45 * const_pi / 180}" effort="176" velocity="${velocity_scale * 110 * const_pi / 180}" />
 			<dynamics friction="10.0" damping="1.0"/>
-			<parent link="${name}_front_harch_link"/>
+			<parent link="${name}_front_arch_link"/>
 			<child link="${name}_roll_link"/>
 		</joint>
@@ -143,5 +143,5 @@
 			<dynamics friction="10.0" damping="1.0"/>
             <mimic joint="${name}_roll_joint" multiplier="1"/>
-			<parent link="${name}_front_harch_link"/>
+			<parent link="${name}_front_arch_link"/>
 			<child link="${name}_front_roll_link"/>
 		</joint>
@@ -149,6 +149,6 @@
 			<inertial>
 				<mass value="${roll_mass}"/>
-				<origin xyz="0 0 0" rpy="0 0 0"/>
-				<cuboid_inertia_def length="0.12" width="0.06" height="0.260" mass="${roll_mass}"/>
+				<origin xyz="0.0010 0 -0.0112" rpy="0 0 0"/>
+				<roll_link_inertia/>
 			</inertial>
 			<visual>
@@ -172,5 +172,5 @@
 			<limit lower="${min_stiffness}" upper="${max_stiffness}" effort="0" velocity="${rate_stiffness}" />
 			<safety_controller soft_lower_limit="${min_stiffness}" soft_upper_limit="${max_stiffness}" k_position="30" k_velocity="30"/>
-			<parent link="${name}_front_harch_link"/>
+			<parent link="${name}_front_arch_link"/>
 			<child link="${name}_front_roll_dummy"/>
 		</joint>
@@ -183,5 +183,5 @@
 			<dynamics friction="10.0" damping="1.0"/>
             <mimic joint="${name}_roll_joint" multiplier="-1"/>
-			<parent link="${name}_back_harch_link"/>
+			<parent link="${name}_back_arch_link"/>
 			<child link="${name}_back_roll_link"/>
 		</joint>
@@ -189,6 +189,6 @@
 			<inertial>
 				<mass value="${roll_mass}"/>
-				<origin xyz="0 0 0" rpy="0 0 0"/>
-				<cuboid_inertia_def length="0.12" width="0.06" height="0.260" mass="${roll_mass}"/>
+				<origin xyz="0.0010 0 -0.0112" rpy="0 0 0"/>
+				<roll_link_inertia/>
 			</inertial>
 			<visual>
@@ -212,5 +212,5 @@
 			<limit lower="${min_stiffness}" upper="${max_stiffness}" effort="0" velocity="${rate_stiffness}" />
 			<safety_controller soft_lower_limit="${min_stiffness}" soft_upper_limit="${max_stiffness}" k_position="30" k_velocity="30"/>
-			<parent link="${name}_back_harch_link"/>
+			<parent link="${name}_back_arch_link"/>
 			<child link="${name}_back_roll_dummy"/>
 		</joint>

Commit message: Corrected stiffness joints

File: softfoot_thing_description/model/softfoot_thing.urdf.xacro (robot description, xacro)
@@ -168,5 +168,5 @@
         <!-- 4) Front roll - stiffness -->
         <joint name="${name}_front_roll_joint_stiffness" type="revolute">
-            <origin xyz="0.058 0 -0.028" rpy="0 0 0"/>
+            <origin xyz="0.058 0 -0.028" rpy="0 -0.1047 0"/>
 			<axis xyz="1 0 0"/>
 			<limit lower="${min_stiffness}" upper="${max_stiffness}" effort="0" velocity="${rate_stiffness}" />
@@ -208,5 +208,5 @@
         <!-- 4) Back roll - stiffness -->
         <joint name="${name}_back_roll_joint_stiffness" type="revolute">
-            <origin xyz="-0.058 0 -0.028" rpy="0 0 ${const_pi}"/>
+            <origin xyz="-0.058 0 -0.028" rpy="0 -0.1047 ${const_pi}"/>
 			<axis xyz="1 0 0"/>
 			<limit lower="${min_stiffness}" upper="${max_stiffness}" effort="0" velocity="${rate_stiffness}" />

Commit message: Still need to add correct collision mesh and dynamic params

File: softfoot_thing_description/model/softfoot_thing.urdf.xacro (robot description, xacro)
@@ -8,7 +8,7 @@
 	<xacro:property name="velocity_scale" value="1"/>
 	<xacro:property name="effort_scale" value="1"/>
-	<xacro:property name="max_stiffness" value="5000"/>
+	<xacro:property name="max_stiffness" value="10"/>
 	<xacro:property name="min_stiffness" value="0"/>
-	<xacro:property name="rate_stiffness" value="20000"/>
+	<xacro:property name="rate_stiffness" value="20"/>
     <!-- Gazebo and Transmission -->
     <!-- Utilities -->
@@ -40,5 +40,5 @@
 				<origin xyz="0 0 0" rpy="0 0 0"/>
 				<geometry>
-					<cylinder radius="0.07" length="0.11"/>
+					<mesh filename="package://softfoot_thing_description/meshes/visual/ankle.stl" scale=" .001 .001 .001"/>
 				</geometry>
 			</collision>
@@ -48,6 +48,6 @@
 			<origin xyz="0 0 0" rpy="0 0 0"/>
 			<axis xyz="0 1 0"/>
-			<limit lower="${-45 * const_pi / 180}" upper="${45 * const_pi / 180}" effort="176" velocity="${velocity_scale * 110 * const_pi / 180}" />
-			<dynamics friction="10.0" damping="1.0"/>
+			<limit lower="${-45 * const_pi / 180}" upper="${45 * const_pi / 180}" effort="10" velocity="${velocity_scale * 45 * const_pi / 180}" />
+			<dynamics friction="1.0" damping="1.0"/>
 			<parent link="${name}_ankle_link"/>
 			<child link="${name}_front_arch_link"/>
@@ -69,5 +69,5 @@
 				<origin xyz="0 0 0.0" rpy="0 0 0"/>
 				<geometry>
-					<sphere radius="0.07"/>
+					<mesh filename="package://softfoot_thing_description/meshes/visual/front_arch_front.stl" scale=" .001 .001 .001"/>
 				</geometry>
 			</collision>
@@ -78,5 +78,5 @@
 			<axis xyz="0 1 0"/>
 			<limit lower="${min_stiffness}" upper="${max_stiffness}" effort="0" velocity="${rate_stiffness}" />
-			<safety_controller soft_lower_limit="${min_stiffness}" soft_upper_limit="${max_stiffness}" k_position="30" k_velocity="30"/>
+			<safety_controller soft_lower_limit="${min_stiffness}" soft_upper_limit="${max_stiffness}" k_position="10" k_velocity="10"/>
 			<parent link="${name}_ankle_link"/>
 			<child link="${name}_front_arch_dummy"/>
@@ -87,6 +87,6 @@
 			<origin xyz="0 0 0" rpy="0 0 0"/>
 			<axis xyz="0 -1 0"/>
-			<limit lower="${-45 * const_pi / 180}" upper="${45 * const_pi / 180}" effort="176" velocity="${velocity_scale * 110 * const_pi / 180}" />
-			<dynamics friction="10.0" damping="1.0"/>
+			<limit lower="${-45 * const_pi / 180}" upper="${45 * const_pi / 180}" effort="10" velocity="${velocity_scale * 45 * const_pi / 180}" />
+			<dynamics friction="1.0" damping="1.0"/>
 			<parent link="${name}_ankle_link"/>
 			<child link="${name}_back_arch_link"/>
@@ -108,5 +108,5 @@
 				<origin xyz="0 0 0" rpy="0 0 0"/>
 				<geometry>
-					<sphere radius="0.07"/>
+					<mesh filename="package://softfoot_thing_description/meshes/visual/front_arch_back.stl" scale=" .001 .001 .001"/>
 				</geometry>
 			</collision>
@@ -117,5 +117,5 @@
 			<axis xyz="0 -1 0"/>
 			<limit lower="${min_stiffness}" upper="${max_stiffness}" effort="0" velocity="${rate_stiffness}" />
-			<safety_controller soft_lower_limit="${min_stiffness}" soft_upper_limit="${max_stiffness}" k_position="30" k_velocity="30"/>
+			<safety_controller soft_lower_limit="${min_stiffness}" soft_upper_limit="${max_stiffness}" k_position="10" k_velocity="10"/>
 			<parent link="${name}_ankle_link"/>
 			<child link="${name}_back_arch_dummy"/>
@@ -126,6 +126,6 @@
 			<origin xyz="0.058 0 -0.028" rpy="0 -0.1047 0"/>
 			<axis xyz="1 0 0"/>
-			<limit lower="${-45 * const_pi / 180}" upper="${45 * const_pi / 180}" effort="176" velocity="${velocity_scale * 110 * const_pi / 180}" />
-			<dynamics friction="10.0" damping="1.0"/>
+			<limit lower="${-45 * const_pi / 180}" upper="${45 * const_pi / 180}" effort="10" velocity="${velocity_scale * 45 * const_pi / 180}" />
+			<dynamics friction="1.0" damping="1.0"/>
 			<parent link="${name}_front_arch_link"/>
 			<child link="${name}_roll_link"/>
@@ -140,6 +140,6 @@
 			<origin xyz="0.058 0 -0.028" rpy="0 -0.1047 0"/>
 			<axis xyz="1 0 0"/>
-			<limit lower="${-45 * const_pi / 180}" upper="${45 * const_pi / 180}" effort="176" velocity="${velocity_scale * 110 * const_pi / 180}" />
-			<dynamics friction="10.0" damping="1.0"/>
+			<limit lower="${-45 * const_pi / 180}" upper="${45 * const_pi / 180}" effort="10" velocity="${velocity_scale * 45 * const_pi / 180}" />
+			<dynamics friction="1.0" damping="1.0"/>
             <mimic joint="${name}_roll_joint" multiplier="1"/>
 			<parent link="${name}_front_arch_link"/>
@@ -162,5 +162,5 @@
 				<origin xyz="0 0 0" rpy="0 0 0"/>
 				<geometry>
-					<sphere radius="0.07"/>
+					<mesh filename="package://softfoot_thing_description/meshes/visual/roll_link_v04.stl" scale=" .001 .001 .001"/>
 				</geometry>
 			</collision>
@@ -171,5 +171,5 @@
 			<axis xyz="1 0 0"/>
 			<limit lower="${min_stiffness}" upper="${max_stiffness}" effort="0" velocity="${rate_stiffness}" />
-			<safety_controller soft_lower_limit="${min_stiffness}" soft_upper_limit="${max_stiffness}" k_position="30" k_velocity="30"/>
+			<safety_controller soft_lower_limit="${min_stiffness}" soft_upper_limit="${max_stiffness}" k_position="10" k_velocity="10"/>
 			<parent link="${name}_front_arch_link"/>
 			<child link="${name}_front_roll_dummy"/>
@@ -180,6 +180,6 @@
 			<origin xyz="-0.058 0 -0.028" rpy="0 -0.1047 ${const_pi}"/>
 			<axis xyz="1 0 0"/>
-			<limit lower="${-45 * const_pi / 180}" upper="${45 * const_pi / 180}" effort="176" velocity="${velocity_scale * 110 * const_pi / 180}" />
-			<dynamics friction="10.0" damping="1.0"/>
+			<limit lower="${-45 * const_pi / 180}" upper="${45 * const_pi / 180}" effort="10" velocity="${velocity_scale * 45 * const_pi / 180}" />
+			<dynamics friction="1.0" damping="1.0"/>
             <mimic joint="${name}_roll_joint" multiplier="-1"/>
 			<parent link="${name}_back_arch_link"/>
@@ -202,5 +202,5 @@
 				<origin xyz="0 0 0" rpy="0 0 0"/>
 				<geometry>
-					<sphere radius="0.07"/>
+					<mesh filename="package://softfoot_thing_description/meshes/visual/roll_link_v04.stl" scale=" .001 .001 .001"/>
 				</geometry>
 			</collision>
@@ -211,5 +211,5 @@
 			<axis xyz="1 0 0"/>
 			<limit lower="${min_stiffness}" upper="${max_stiffness}" effort="0" velocity="${rate_stiffness}" />
-			<safety_controller soft_lower_limit="${min_stiffness}" soft_upper_limit="${max_stiffness}" k_position="30" k_velocity="30"/>
+			<safety_controller soft_lower_limit="${min_stiffness}" soft_upper_limit="${max_stiffness}" k_position="10" k_velocity="10"/>
 			<parent link="${name}_back_arch_link"/>
 			<child link="${name}_back_roll_dummy"/>

Commit message: Added leg to robot and adjusted urdf model accordingly

File: softfoot_thing_description/model/softfoot_thing.urdf.xacro (robot description, xacro)
@@ -19,9 +19,16 @@
 	<!-- URDF -->
 	<xacro:macro name="softfoot_thing" params="parent name *origin">
-		<!-- 1) Ankle of the foot - fixed to parent. -->
-		<joint name="${parent}_${name}_ankle_joint" type="fixed">
+		<!-- 0) Ankle base - fixed to parent. -->
+		<joint name="${parent}_${name}_ankle_base_joint" type="fixed">
 			<xacro:insert_block name="origin"/>
 			<origin xyz="0 0 0" rpy="0 0 0"/>
 			<parent link="${parent}"/>
+			<child link="${name}_ankle_base_link"/>
+		</joint>
+		<link name="${name}_ankle_base_link"/>
+		<!-- 1) Ankle of the foot - fixed to parent. -->
+		<joint name="${name}_ankle_joint" type="fixed">
+			<origin xyz="0 0 -0.022" rpy="0 0 0"/>
+			<parent link="${name}_ankle_base_link"/>
 			<child link="${name}_ankle_link"/>
 		</joint>
@@ -69,5 +76,5 @@
 			</visual>
 			<collision>
-				<origin xyz="0 0 0.0" rpy="0 0 0"/>
+				<origin xyz="0 0 0" rpy="0 0 0"/>
 				<geometry>
 					<mesh filename="package://softfoot_thing_description/meshes/visual/front_arch_front.stl" scale=" .001 .001 .001"/>

File: softfoot_thing_description/robot/pisa_softfoot.urdf.xacro (robot description, xacro)
@@ -6,7 +6,19 @@
   <!-- WORLD -->
   <link name="world"/>
+  <!-- LEG -->
+  <joint name="world_to_leg" type="fixed">
+    <parent link="world"/>
+    <child link="leg_link"/>
+  </joint>
+  <link name="leg_link">
+    <visual>
+      <geometry>
+        <cylinder length="0.1" radius="0.015"/>
+      </geometry>
+    </visual>
+  </link>
   <!-- FOOT -->
-  <xacro:softfoot_thing name="pisa_softfoot" parent="world">
-    <origin xyz="0 0 0" rpy="0 0 0"/>
+  <xacro:softfoot_thing name="pisa_softfoot" parent="leg_link">
+    <origin xyz="0 0 -0.05" rpy="0 0 0"/>
   </xacro:softfoot_thing>
 </robot>

Commit message: Added nive visualization materials

File: softfoot_thing_description/model/softfoot_thing.urdf.xacro (robot description, xacro)
@@ -44,5 +44,5 @@
 					<mesh filename="package://softfoot_thing_description/meshes/visual/ankle.stl" scale=" .001 .001 .001"/>
 				</geometry>
-				<material name="SoftFoot/Silver"/>
+				<material name="SoftFoot/Grey"/>
 			</visual>
 			<collision>
@@ -73,5 +73,5 @@
 					<mesh filename="package://softfoot_thing_description/meshes/visual/front_arch_front.stl" scale=" .001 .001 .001"/>
 				</geometry>
-				<material name="SoftFoot/Silver"/>
+				<material name="SoftFoot/Grey"/>
 			</visual>
 			<collision>
@@ -112,5 +112,5 @@
 					<mesh filename="package://softfoot_thing_description/meshes/visual/front_arch_back.stl" scale=" .001 .001 .001"/>
 				</geometry>
-				<material name="SoftFoot/Silver"/>
+				<material name="SoftFoot/Grey"/>
 			</visual>
 			<collision>
@@ -166,5 +166,5 @@
 					<mesh filename="package://softfoot_thing_description/meshes/visual/roll_link_v04.stl" scale=" .001 .001 .001"/>
 				</geometry>
-				<material name="SoftFoot/Silver"/>
+				<material name="SoftFoot/Grey"/>
 			</visual>
 			<collision>
@@ -206,5 +206,5 @@
 					<mesh filename="package://softfoot_thing_description/meshes/visual/roll_link_v04.stl" scale=" .001 .001 .001"/>
 				</geometry>
-				<material name="SoftFoot/Silver"/>
+				<material name="SoftFoot/Grey"/>
 			</visual>
 			<collision>

File: softfoot_thing_description/robot/pisa_softfoot.urdf.xacro (robot description, xacro)
@@ -16,4 +16,8 @@
         <cylinder length="0.1" radius="0.015"/>
       </geometry>
+      <material name="material.metal">
+        <texture />
+        <color rgba="0.1 0.1 0.1 1" />
+      </material>
     </visual>
   </link>

Commit message: Mimic also stiffness

File: softfoot_thing_description/model/softfoot_thing.urdf.xacro (robot description, xacro)
@@ -180,4 +180,5 @@
 			<axis xyz="1 0 0"/>
 			<limit lower="${min_stiffness}" upper="${max_stiffness}" effort="0" velocity="${rate_stiffness}" />
+			<mimic joint="${name}_roll_joint" multiplier="1"/>
 			<safety_controller soft_lower_limit="${min_stiffness}" soft_upper_limit="${max_stiffness}" k_position="10" k_velocity="10"/>
 			<parent link="${name}_front_arch_link"/>
@@ -220,4 +221,5 @@
 			<axis xyz="1 0 0"/>
 			<limit lower="${min_stiffness}" upper="${max_stiffness}" effort="0" velocity="${rate_stiffness}" />
+			<mimic joint="${name}_roll_joint" multiplier="-1"/>
 			<safety_controller soft_lower_limit="${min_stiffness}" soft_upper_limit="${max_stiffness}" k_position="10" k_velocity="10"/>
 			<parent link="${name}_back_arch_link"/>
