Commit message: Retuning to make simulation work

File: softfoot_thing_description/model/softfoot_thing.urdf.xacro (robot description, xacro)
@@ -26,5 +26,9 @@
 			<child link="${name}_ankle_base_link"/>
 		</joint>
-		<link name="${name}_ankle_base_link"/>
+		<link name="${name}_ankle_base_link">
+			<inertial>
+				<xacro:insert_block name="negligible_inertia"/>
+			</inertial>
+		</link>
 		<!-- 1) Ankle of the foot - fixed to parent. -->
 		<joint name="${name}_ankle_joint" type="fixed">
@@ -57,6 +61,6 @@
 			<origin xyz="0 0 0" rpy="0 0 0"/>
 			<axis xyz="0 1 0"/>
-			<limit lower="${-45 * const_pi / 180}" upper="${45 * const_pi / 180}" effort="10" velocity="${velocity_scale * 45 * const_pi / 180}" />
-			<dynamics friction="1.0" damping="1.0"/>
+			<limit lower="${-45 * const_pi / 180}" upper="${45 * const_pi / 180}" effort="1" velocity="${velocity_scale * 45 * const_pi / 180}" />
+			<dynamics friction="0.01" damping="0.01"/>
 			<parent link="${name}_ankle_link"/>
 			<child link="${name}_front_arch_link"/>
@@ -83,5 +87,5 @@
 		</link>
         <!-- 2) Front arch - stiffness -->
-        <joint name="${name}_front_arch_joint_stiffness" type="revolute">
+        <!-- <joint name="${name}_front_arch_joint_stiffness" type="revolute">
             <origin xyz="0 0 0" rpy="0 0 0"/>
 			<axis xyz="0 1 0"/>
@@ -91,11 +95,11 @@
 			<child link="${name}_front_arch_dummy"/>
 		</joint>
-		<link name="${name}_front_arch_dummy"/>
+		<link name="${name}_front_arch_dummy"/> -->
         <!-- 3) Back arch - joint along y-axis to pitch -->
 		<joint name="${name}_back_arch_joint" type="revolute">
 			<origin xyz="0 0 0" rpy="0 0 0"/>
 			<axis xyz="0 -1 0"/>
-			<limit lower="${-45 * const_pi / 180}" upper="${45 * const_pi / 180}" effort="10" velocity="${velocity_scale * 45 * const_pi / 180}" />
-			<dynamics friction="1.0" damping="1.0"/>
+			<limit lower="${-45 * const_pi / 180}" upper="${45 * const_pi / 180}" effort="1" velocity="${velocity_scale * 45 * const_pi / 180}" />
+			<dynamics friction="0.01" damping="0.01"/>
 			<parent link="${name}_ankle_link"/>
 			<child link="${name}_back_arch_link"/>
@@ -122,5 +126,5 @@
 		</link>
         <!-- 3) Back arch - stiffness -->
-        <joint name="${name}_back_arch_joint_stiffness" type="revolute">
+        <!-- <joint name="${name}_back_arch_joint_stiffness" type="revolute">
             <origin xyz="0 0 0" rpy="0 0 0"/>
 			<axis xyz="0 -1 0"/>
@@ -130,11 +134,11 @@
 			<child link="${name}_back_arch_dummy"/>
 		</joint>
-		<link name="${name}_back_arch_dummy"/>
+		<link name="${name}_back_arch_dummy"/> -->
         <!-- x) Roll driving joint - we suppose the roll joints move specularly -->
 		<joint name="${name}_roll_joint" type="revolute">
 			<origin xyz="0.058 0 -0.028" rpy="0 -0.1047 0"/>
 			<axis xyz="1 0 0"/>
-			<limit lower="${-45 * const_pi / 180}" upper="${45 * const_pi / 180}" effort="10" velocity="${velocity_scale * 45 * const_pi / 180}" />
-			<dynamics friction="1.0" damping="1.0"/>
+			<limit lower="${-45 * const_pi / 180}" upper="${45 * const_pi / 180}" effort="1" velocity="${velocity_scale * 45 * const_pi / 180}" />
+			<dynamics friction="0.01" damping="0.01"/>
 			<parent link="${name}_front_arch_link"/>
 			<child link="${name}_roll_link"/>
@@ -149,6 +153,6 @@
 			<origin xyz="0.058 0 -0.028" rpy="0 -0.1047 0"/>
 			<axis xyz="1 0 0"/>
-			<limit lower="${-45 * const_pi / 180}" upper="${45 * const_pi / 180}" effort="10" velocity="${velocity_scale * 45 * const_pi / 180}" />
-			<dynamics friction="1.0" damping="1.0"/>
+			<limit lower="${-45 * const_pi / 180}" upper="${45 * const_pi / 180}" effort="1" velocity="${velocity_scale * 45 * const_pi / 180}" />
+			<dynamics friction="0.01" damping="0.01"/>
             <mimic joint="${name}_roll_joint" multiplier="1"/>
 			<parent link="${name}_front_arch_link"/>
@@ -176,5 +180,5 @@
 		</link>
         <!-- 4) Front roll - stiffness -->
-        <joint name="${name}_front_roll_joint_stiffness" type="revolute">
+        <!-- <joint name="${name}_front_roll_joint_stiffness" type="revolute">
             <origin xyz="0.058 0 -0.028" rpy="0 -0.1047 0"/>
 			<axis xyz="1 0 0"/>
@@ -185,11 +189,11 @@
 			<child link="${name}_front_roll_dummy"/>
 		</joint>
-		<link name="${name}_front_roll_dummy"/>
+		<link name="${name}_front_roll_dummy"/> -->
         <!-- 4) Back roll - joint along x-axis to roll -->
 		<joint name="${name}_back_roll_joint" type="revolute">
 			<origin xyz="-0.058 0 -0.028" rpy="0 -0.1047 ${const_pi}"/>
 			<axis xyz="1 0 0"/>
-			<limit lower="${-45 * const_pi / 180}" upper="${45 * const_pi / 180}" effort="10" velocity="${velocity_scale * 45 * const_pi / 180}" />
-			<dynamics friction="1.0" damping="1.0"/>
+			<limit lower="${-45 * const_pi / 180}" upper="${45 * const_pi / 180}" effort="1" velocity="${velocity_scale * 45 * const_pi / 180}" />
+			<dynamics friction="0.01" damping="0.01"/>
             <mimic joint="${name}_roll_joint" multiplier="-1"/>
 			<parent link="${name}_back_arch_link"/>
@@ -217,5 +221,5 @@
 		</link>
         <!-- 4) Back roll - stiffness -->
-        <joint name="${name}_back_roll_joint_stiffness" type="revolute">
+        <!-- <joint name="${name}_back_roll_joint_stiffness" type="revolute">
             <origin xyz="-0.058 0 -0.028" rpy="0 -0.1047 ${const_pi}"/>
 			<axis xyz="1 0 0"/>
@@ -226,5 +230,5 @@
 			<child link="${name}_back_roll_dummy"/>
 		</joint>
-		<link name="${name}_back_roll_dummy"/>
+		<link name="${name}_back_roll_dummy"/> -->
 		<!-- Gazebo elements -->
 		<xacro:softfoot_thing_gazebo name="${name}"/>

File: softfoot_thing_description/robot/pisa_softfoot.urdf.xacro (robot description, xacro)
@@ -8,4 +8,5 @@
   <!-- LEG -->
   <joint name="world_to_leg" type="fixed">
+    <origin xyz="0 0 0.2" rpy="0 0 0"/>
     <parent link="world"/>
     <child link="leg_link"/>

Commit message: Simulation seems better but still grey

File: softfoot_thing_description/model/softfoot_thing.urdf.xacro (robot description, xacro)
@@ -61,5 +61,5 @@
 			<origin xyz="0 0 0" rpy="0 0 0"/>
 			<axis xyz="0 1 0"/>
-			<limit lower="${-45 * const_pi / 180}" upper="${45 * const_pi / 180}" effort="1" velocity="${velocity_scale * 45 * const_pi / 180}" />
+			<limit lower="${-45 * const_pi / 180}" upper="${45 * const_pi / 180}" effort="1" velocity="1" />
 			<dynamics friction="0.01" damping="0.01"/>
 			<parent link="${name}_ankle_link"/>
@@ -100,5 +100,5 @@
 			<origin xyz="0 0 0" rpy="0 0 0"/>
 			<axis xyz="0 -1 0"/>
-			<limit lower="${-45 * const_pi / 180}" upper="${45 * const_pi / 180}" effort="1" velocity="${velocity_scale * 45 * const_pi / 180}" />
+			<limit lower="${-45 * const_pi / 180}" upper="${45 * const_pi / 180}" effort="1" velocity="1" />
 			<dynamics friction="0.01" damping="0.01"/>
 			<parent link="${name}_ankle_link"/>
@@ -139,5 +139,5 @@
 			<origin xyz="0.058 0 -0.028" rpy="0 -0.1047 0"/>
 			<axis xyz="1 0 0"/>
-			<limit lower="${-45 * const_pi / 180}" upper="${45 * const_pi / 180}" effort="1" velocity="${velocity_scale * 45 * const_pi / 180}" />
+			<limit lower="${-45 * const_pi / 180}" upper="${45 * const_pi / 180}" effort="1" velocity="1" />
 			<dynamics friction="0.01" damping="0.01"/>
 			<parent link="${name}_front_arch_link"/>
@@ -153,6 +153,6 @@
 			<origin xyz="0.058 0 -0.028" rpy="0 -0.1047 0"/>
 			<axis xyz="1 0 0"/>
-			<limit lower="${-45 * const_pi / 180}" upper="${45 * const_pi / 180}" effort="1" velocity="${velocity_scale * 45 * const_pi / 180}" />
-			<dynamics friction="0.01" damping="0.01"/>
+			<limit lower="${-45 * const_pi / 180}" upper="${45 * const_pi / 180}" effort="1" velocity="1" />
+			<dynamics friction="0.0001" damping="0.0001"/>
             <!-- <mimic joint="${name}_roll_joint" multiplier="1"/> -->
 			<parent link="${name}_front_arch_link"/>
@@ -194,6 +194,6 @@
 			<origin xyz="-0.058 0 -0.028" rpy="0 -0.1047 ${const_pi}"/>
 			<axis xyz="1 0 0"/>
-			<limit lower="${-45 * const_pi / 180}" upper="${45 * const_pi / 180}" effort="1" velocity="${velocity_scale * 45 * const_pi / 180}" />
-			<dynamics friction="0.01" damping="0.01"/>
+			<limit lower="${-45 * const_pi / 180}" upper="${45 * const_pi / 180}" effort="1" velocity="1" />
+			<dynamics friction="0.0001" damping="0.0001"/>
             <!-- <mimic joint="${name}_roll_joint" multiplier="-1"/> -->
 			<parent link="${name}_back_arch_link"/>

Commit message: Restored mimic joint

File: softfoot_thing_description/model/softfoot_thing.urdf.xacro (robot description, xacro)
@@ -155,5 +155,5 @@
 			<limit lower="${-45 * const_pi / 180}" upper="${45 * const_pi / 180}" effort="1" velocity="1" />
 			<dynamics friction="0.0001" damping="0.0001"/>
-            <!-- <mimic joint="${name}_roll_joint" multiplier="1"/> -->
+            <mimic joint="${name}_roll_joint" multiplier="1"/>
 			<parent link="${name}_front_arch_link"/>
 			<child link="${name}_front_roll_link"/>
@@ -196,5 +196,5 @@
 			<limit lower="${-45 * const_pi / 180}" upper="${45 * const_pi / 180}" effort="1" velocity="1" />
 			<dynamics friction="0.0001" damping="0.0001"/>
-            <!-- <mimic joint="${name}_roll_joint" multiplier="-1"/> -->
+            <mimic joint="${name}_roll_joint" multiplier="-1"/>
 			<parent link="${name}_back_arch_link"/>
 			<child link="${name}_back_roll_link"/>

Commit message: Added all central chain to urdf

File: softfoot_thing_description/model/softfoot_thing.urdf.xacro (robot description, xacro)
@@ -15,4 +15,5 @@
 	<xacro:include filename="$(find softfoot_thing_description)/model/softfoot_thing.transmission.xacro"/>
     <!-- Utilities -->
+	<xacro:include filename="$(find softfoot_thing_description)/model/chain_thing.urdf.xacro"/>
     <xacro:include filename="$(find softfoot_thing_description)/model/softfoot_thing_inertia.xacro"/>
     <xacro:include filename="$(find softfoot_thing_description)/model/softfoot_thing_materials.xacro"/>
@@ -231,4 +232,9 @@
 		</joint>
 		<link name="${name}_back_roll_dummy"/> -->
+		<!-- 5) Chain - joints along y-axis to pitch -->
+		<xacro:chain_thing name="middle_chain" parent="${name}_front_roll_link">
+    		<!-- <origin xyz="-0.00209969 0 -0.0118454" rpy="0 0.1046328 0"/> -->
+			<origin xyz="-0.00209969 0 -0.0118454" rpy="${-(const_pi / 2) + 0.1046328} 0 ${const_pi / 2}"/>
+  		</xacro:chain_thing>
 		<!-- Gazebo elements -->
 		<xacro:softfoot_thing_gazebo name="${name}"/>

Commit message: Specified that the insertion point is for middle chain

File: softfoot_thing_description/model/softfoot_thing.urdf.xacro (robot description, xacro)
@@ -232,11 +232,11 @@
 		</joint>
 		<link name="${name}_back_roll_dummy"/> -->
-		<!-- 5) Chain insertion point -->
-        <joint name="${name}_chain_insertion_joint" type="fixed">
+		<!-- 5) Middle chain insertion point -->
+        <joint name="${name}_middle_chain_insertion_joint" type="fixed">
 			<origin xyz="-0.00209969 0 -0.0118454" rpy="${-(const_pi / 2) - 0.105} 0 ${-const_pi / 2}"/>
 			<parent link="${name}_back_roll_link"/>
-			<child link="${name}_chain_insertion_link"/>
-		</joint>
-		<link name="${name}_chain_insertion_link"/>
+			<child link="${name}_middle_chain_insertion_link"/>
+		</joint>
+		<link name="${name}_middle_chain_insertion_link"/>
 		<!-- 6) Chain - starting from front -->
 		<xacro:chain_thing name="middle_chain" foot="${name}" parent="${name}_front_roll_link">

Commit message: Arch joint limits to slightly more realistic values

File: softfoot_thing_description/model/softfoot_thing.urdf.xacro (robot description, xacro)
@@ -62,5 +62,5 @@
 			<origin xyz="0 0 0" rpy="0 0 0"/>
 			<axis xyz="0 1 0"/>
-			<limit lower="${-45 * const_pi / 180}" upper="${45 * const_pi / 180}" effort="1" velocity="1" />
+			<limit lower="${-30 * const_pi / 180}" upper="${30 * const_pi / 180}" effort="1" velocity="1" />
 			<dynamics friction="0.01" damping="0.01"/>
 			<parent link="${name}_ankle_link"/>
@@ -101,5 +101,5 @@
 			<origin xyz="0 0 0" rpy="0 0 0"/>
 			<axis xyz="0 -1 0"/>
-			<limit lower="${-45 * const_pi / 180}" upper="${45 * const_pi / 180}" effort="1" velocity="1" />
+			<limit lower="${-30 * const_pi / 180}" upper="${30 * const_pi / 180}" effort="1" velocity="1" />
 			<dynamics friction="0.01" damping="0.01"/>
 			<parent link="${name}_ankle_link"/>

Commit message: More realistic limits and coupling, conversion error corrected and code clean up

File: softfoot_thing_description/model/softfoot_thing.urdf.xacro (robot description, xacro)
@@ -62,5 +62,5 @@
 			<origin xyz="0 0 0" rpy="0 0 0"/>
 			<axis xyz="0 1 0"/>
-			<limit lower="${-30 * const_pi / 180}" upper="${30 * const_pi / 180}" effort="1" velocity="1" />
+			<limit lower="${-30 * const_pi / 180}" upper="${60 * const_pi / 180}" effort="1" velocity="1" />
 			<dynamics friction="0.01" damping="0.01"/>
 			<parent link="${name}_ankle_link"/>
@@ -101,5 +101,5 @@
 			<origin xyz="0 0 0" rpy="0 0 0"/>
 			<axis xyz="0 -1 0"/>
-			<limit lower="${-30 * const_pi / 180}" upper="${30 * const_pi / 180}" effort="1" velocity="1" />
+			<limit lower="${-30 * const_pi / 180}" upper="${60 * const_pi / 180}" effort="1" velocity="1" />
 			<dynamics friction="0.01" damping="0.01"/>
 			<parent link="${name}_ankle_link"/>

Commit message: Not realistic inertia on roll link was creating imbalance

File: softfoot_thing_description/model/softfoot_thing.urdf.xacro (robot description, xacro)
@@ -146,8 +146,8 @@
 		</joint>
         <link name="${name}_roll_link">
-			<inertial>
-				<xacro:insert_block name="negligible_inertia"/>
-			</inertial>
-		</link>
+                        <inertial>
+                                <xacro:insert_block name="really_negligible_inertia"/>
+                        </inertial>
+                </link>
         <!-- 4) Front roll - joint along x-axis to roll -->
 		<joint name="${name}_front_roll_joint" type="revolute">

File: softfoot_thing_description/model/softfoot_thing_inertia.xacro (robot description, xacro)
@@ -2,4 +2,5 @@
 <robot xmlns:xacro="http://www.ros.org/wiki/xacro">
   <xacro:property name="negligible_mass" value="0.1"/>
+  <xacro:property name="really_negligible_mass" value="0.00001"/>
   <xacro:property name="mm2tom2" value="0.000001"/>
   <!-- INERTIA MATRICES FOR LINKS (wrt frames in urdf inertial) -->
@@ -45,3 +46,9 @@
                 ixy="0.0" ixz="0.0" iyz="0.0"/>
   </xacro:property>
+<xacro:property name="really_negligible_inertia">
+    <origin xyz="0 0 0"/>
+    <mass value="${really_negligible_mass}"/>
+    <inertia  ixx="${mm2tom2 * 0.00001}" iyy="${mm2tom2 * 0.00001}" izz="${mm2tom2 * 0.00001}"
+              ixy="0.0" ixz="0.0" iyz="0.0"/>
+  </xacro:property>
 </robot>

Commit message: More realistic friction and damping

File: softfoot_thing_description/model/softfoot_thing.urdf.xacro (robot description, xacro)
@@ -63,5 +63,5 @@
 			<axis xyz="0 1 0"/>
 			<limit lower="${-30 * const_pi / 180}" upper="${60 * const_pi / 180}" effort="1" velocity="1" />
-			<dynamics friction="0.01" damping="0.01"/>
+                        <dynamics friction="0.0001" damping="0.0001"/>
 			<parent link="${name}_ankle_link"/>
 			<child link="${name}_front_arch_link"/>
@@ -102,5 +102,5 @@
 			<axis xyz="0 -1 0"/>
 			<limit lower="${-30 * const_pi / 180}" upper="${60 * const_pi / 180}" effort="1" velocity="1" />
-			<dynamics friction="0.01" damping="0.01"/>
+                        <dynamics friction="0.0001" damping="0.0001"/>
 			<parent link="${name}_ankle_link"/>
 			<child link="${name}_back_arch_link"/>
