Commit message: Better names for chain elements and gazebo references

File: softfoot_thing_description/model/chain_thing.urdf.xacro (robot description, xacro)
@@ -11,16 +11,16 @@
     <xacro:include filename="$(find softfoot_thing_description)/model/chain_thing_materials.xacro"/>
 	<!-- URDF -->
-	<xacro:macro name="chain_thing" params="parent name *origin">
+	<xacro:macro name="chain_thing" params="parent name foot *origin">
 		<!-- 0) Chain 1 - joint along y-axis to pitch -->
-		<joint name="${parent}_${name}_1_joint" type="revolute">
+		<joint name="${foot}_${name}_1_joint" type="revolute">
 			<xacro:insert_block name="origin"/>
 			<origin xyz="0 0 0" rpy="0 0 0"/>
 			<axis xyz="0 1 0"/>
 			<limit lower="${-45 * const_pi / 180}" upper="${45 * const_pi / 180}" effort="1" velocity="1" />
-			<dynamics friction="0.01" damping="0.01"/>
+			<dynamics friction="0.0001" damping="0.0001"/>
 			<parent link="${parent}"/>
-			<child link="${parent}_${name}_1_link"/>
-		</joint>
-		<link name="${parent}_${name}_1_link">
+			<child link="${foot}_${name}_1_link"/>
+		</joint>
+		<link name="${foot}_${name}_1_link">
 			<inertial>
 				<mass value="${inner_chain_mass}"/>
@@ -43,13 +43,13 @@
 		</link>
 		<!-- 1) Chain 2 - joint along y-axis to pitch -->
-		<joint name="${parent}_${name}_2_joint" type="revolute">
-			<origin xyz="0 0 0.0127" rpy="0 0 0"/>
-			<axis xyz="0 1 0"/>
-			<limit lower="${-45 * const_pi / 180}" upper="${45 * const_pi / 180}" effort="1" velocity="1" />
-			<dynamics friction="0.01" damping="0.01"/>
-			<parent link="${parent}_${name}_1_link"/>
-			<child link="${parent}_${name}_2_link"/>
-		</joint>
-		<link name="${parent}_${name}_2_link">
+		<joint name="${foot}_${name}_2_joint" type="revolute">
+			<origin xyz="0 0 0.0127" rpy="0 0 0"/>
+			<axis xyz="0 1 0"/>
+			<limit lower="${-45 * const_pi / 180}" upper="${45 * const_pi / 180}" effort="1" velocity="1" />
+			<dynamics friction="0.0001" damping="0.0001"/>
+			<parent link="${foot}_${name}_1_link"/>
+			<child link="${foot}_${name}_2_link"/>
+		</joint>
+		<link name="${foot}_${name}_2_link">
 			<inertial>
 				<mass value="${outer_chain_mass}"/>
@@ -72,13 +72,13 @@
 		</link>
 		<!-- 2) Chain 3 - joint along y-axis to pitch -->
-		<joint name="${parent}_${name}_3_joint" type="revolute">
-			<origin xyz="0 0 0.0127" rpy="0 0 0"/>
-			<axis xyz="0 1 0"/>
-			<limit lower="${-45 * const_pi / 180}" upper="${45 * const_pi / 180}" effort="1" velocity="1" />
-			<dynamics friction="0.01" damping="0.01"/>
-			<parent link="${parent}_${name}_2_link"/>
-			<child link="${parent}_${name}_3_link"/>
-		</joint>
-		<link name="${parent}_${name}_3_link">
+		<joint name="${foot}_${name}_3_joint" type="revolute">
+			<origin xyz="0 0 0.0127" rpy="0 0 0"/>
+			<axis xyz="0 1 0"/>
+			<limit lower="${-45 * const_pi / 180}" upper="${45 * const_pi / 180}" effort="1" velocity="1" />
+			<dynamics friction="0.0001" damping="0.0001"/>
+			<parent link="${foot}_${name}_2_link"/>
+			<child link="${foot}_${name}_3_link"/>
+		</joint>
+		<link name="${foot}_${name}_3_link">
 			<inertial>
 				<mass value="${inner_chain_mass}"/>
@@ -101,13 +101,13 @@
 		</link>
 		<!-- 3) Chain 4 - joint along y-axis to pitch -->
-		<joint name="${parent}_${name}_4_joint" type="revolute">
-			<origin xyz="0 0 0.0127" rpy="0 0 0"/>
-			<axis xyz="0 1 0"/>
-			<limit lower="${-45 * const_pi / 180}" upper="${45 * const_pi / 180}" effort="1" velocity="1" />
-			<dynamics friction="0.01" damping="0.01"/>
-			<parent link="${parent}_${name}_3_link"/>
-			<child link="${parent}_${name}_4_link"/>
-		</joint>
-		<link name="${parent}_${name}_4_link">
+		<joint name="${foot}_${name}_4_joint" type="revolute">
+			<origin xyz="0 0 0.0127" rpy="0 0 0"/>
+			<axis xyz="0 1 0"/>
+			<limit lower="${-45 * const_pi / 180}" upper="${45 * const_pi / 180}" effort="1" velocity="1" />
+			<dynamics friction="0.0001" damping="0.0001"/>
+			<parent link="${foot}_${name}_3_link"/>
+			<child link="${foot}_${name}_4_link"/>
+		</joint>
+		<link name="${foot}_${name}_4_link">
 			<inertial>
 				<mass value="${outer_chain_mass}"/>
@@ -130,13 +130,13 @@
 		</link>
 		<!-- 4) Chain 5 - joint along y-axis to pitch -->
-		<joint name="${parent}_${name}_5_joint" type="revolute">
-			<origin xyz="0 0 0.0127" rpy="0 0 0"/>
-			<axis xyz="0 1 0"/>
-			<limit lower="${-45 * const_pi / 180}" upper="${45 * const_pi / 180}" effort="1" velocity="1" />
-			<dynamics friction="0.01" damping="0.01"/>
-			<parent link="${parent}_${name}_4_link"/>
-			<child link="${parent}_${name}_5_link"/>
-		</joint>
-		<link name="${parent}_${name}_5_link">
+		<joint name="${foot}_${name}_5_joint" type="revolute">
+			<origin xyz="0 0 0.0127" rpy="0 0 0"/>
+			<axis xyz="0 1 0"/>
+			<limit lower="${-45 * const_pi / 180}" upper="${45 * const_pi / 180}" effort="1" velocity="1" />
+			<dynamics friction="0.0001" damping="0.0001"/>
+			<parent link="${foot}_${name}_4_link"/>
+			<child link="${foot}_${name}_5_link"/>
+		</joint>
+		<link name="${foot}_${name}_5_link">
 			<inertial>
 				<mass value="${inner_chain_mass}"/>
@@ -159,13 +159,13 @@
 		</link>
 		<!-- 5) Chain 6 - joint along y-axis to pitch -->
-		<joint name="${parent}_${name}_6_joint" type="revolute">
-			<origin xyz="0 0 0.0127" rpy="0 0 0"/>
-			<axis xyz="0 1 0"/>
-			<limit lower="${-45 * const_pi / 180}" upper="${45 * const_pi / 180}" effort="1" velocity="1" />
-			<dynamics friction="0.01" damping="0.01"/>
-			<parent link="${parent}_${name}_5_link"/>
-			<child link="${parent}_${name}_6_link"/>
-		</joint>
-		<link name="${parent}_${name}_6_link">
+		<joint name="${foot}_${name}_6_joint" type="revolute">
+			<origin xyz="0 0 0.0127" rpy="0 0 0"/>
+			<axis xyz="0 1 0"/>
+			<limit lower="${-45 * const_pi / 180}" upper="${45 * const_pi / 180}" effort="1" velocity="1" />
+			<dynamics friction="0.0001" damping="0.0001"/>
+			<parent link="${foot}_${name}_5_link"/>
+			<child link="${foot}_${name}_6_link"/>
+		</joint>
+		<link name="${foot}_${name}_6_link">
 			<inertial>
 				<mass value="${outer_chain_mass}"/>
@@ -188,13 +188,13 @@
 		</link>
 		<!-- 6) Chain 7 - joint along y-axis to pitch -->
-		<joint name="${parent}_${name}_7_joint" type="revolute">
-			<origin xyz="0 0 0.0127" rpy="0 0 0"/>
-			<axis xyz="0 1 0"/>
-			<limit lower="${-45 * const_pi / 180}" upper="${45 * const_pi / 180}" effort="1" velocity="1" />
-			<dynamics friction="0.01" damping="0.01"/>
-			<parent link="${parent}_${name}_6_link"/>
-			<child link="${parent}_${name}_7_link"/>
-		</joint>
-		<link name="${parent}_${name}_7_link">
+		<joint name="${foot}_${name}_7_joint" type="revolute">
+			<origin xyz="0 0 0.0127" rpy="0 0 0"/>
+			<axis xyz="0 1 0"/>
+			<limit lower="${-45 * const_pi / 180}" upper="${45 * const_pi / 180}" effort="1" velocity="1" />
+			<dynamics friction="0.0001" damping="0.0001"/>
+			<parent link="${foot}_${name}_6_link"/>
+			<child link="${foot}_${name}_7_link"/>
+		</joint>
+		<link name="${foot}_${name}_7_link">
 			<inertial>
 				<mass value="${inner_chain_mass}"/>
@@ -217,13 +217,13 @@
 		</link>
 		<!-- 7) Chain 8 - joint along y-axis to pitch -->
-		<joint name="${parent}_${name}_8_joint" type="revolute">
-			<origin xyz="0 0 0.0127" rpy="0 0 0"/>
-			<axis xyz="0 1 0"/>
-			<limit lower="${-45 * const_pi / 180}" upper="${45 * const_pi / 180}" effort="1" velocity="1" />
-			<dynamics friction="0.01" damping="0.01"/>
-			<parent link="${parent}_${name}_7_link"/>
-			<child link="${parent}_${name}_8_link"/>
-		</joint>
-		<link name="${parent}_${name}_8_link">
+		<joint name="${foot}_${name}_8_joint" type="revolute">
+			<origin xyz="0 0 0.0127" rpy="0 0 0"/>
+			<axis xyz="0 1 0"/>
+			<limit lower="${-45 * const_pi / 180}" upper="${45 * const_pi / 180}" effort="1" velocity="1" />
+			<dynamics friction="0.0001" damping="0.0001"/>
+			<parent link="${foot}_${name}_7_link"/>
+			<child link="${foot}_${name}_8_link"/>
+		</joint>
+		<link name="${foot}_${name}_8_link">
 			<inertial>
 				<mass value="${outer_chain_mass}"/>
@@ -246,13 +246,13 @@
 		</link>
 		<!-- 8) Chain 9 - joint along y-axis to pitch -->
-		<joint name="${parent}_${name}_9_joint" type="revolute">
-			<origin xyz="0 0 0.0127" rpy="0 0 0"/>
-			<axis xyz="0 1 0"/>
-			<limit lower="${-45 * const_pi / 180}" upper="${45 * const_pi / 180}" effort="1" velocity="1" />
-			<dynamics friction="0.01" damping="0.01"/>
-			<parent link="${parent}_${name}_8_link"/>
-			<child link="${parent}_${name}_9_link"/>
-		</joint>
-		<link name="${parent}_${name}_9_link">
+		<joint name="${foot}_${name}_9_joint" type="revolute">
+			<origin xyz="0 0 0.0127" rpy="0 0 0"/>
+			<axis xyz="0 1 0"/>
+			<limit lower="${-45 * const_pi / 180}" upper="${45 * const_pi / 180}" effort="1" velocity="1" />
+			<dynamics friction="0.0001" damping="0.0001"/>
+			<parent link="${foot}_${name}_8_link"/>
+			<child link="${foot}_${name}_9_link"/>
+		</joint>
+		<link name="${foot}_${name}_9_link">
 			<inertial>
 				<mass value="${inner_chain_mass}"/>

File: softfoot_thing_description/model/softfoot_thing.gazebo.xacro (robot description, xacro)
@@ -1,5 +1,5 @@
 <?xml version="1.0"?>
 <robot xmlns:xacro="http://www.ros.org/wiki/xacro">
-	<xacro:macro name="softfoot_thing_gazebo" params="name">
+	<xacro:macro name="softfoot_thing_gazebo" params="name chain_name">
 		<!-- Ros control (For future actuated case) -->
 		<!-- <gazebo>
@@ -18,9 +18,17 @@
        		<plugin name="joint_state_publisher" filename="libgazebo_ros_joint_state_publisher.so">
          		<robotNamespace>${name}</robotNamespace>
-         		<jointName>${name}_front_arch_joint, ${name}_back_arch_joint, ${name}_roll_joint, ${name}_front_roll_joint, ${name}_back_roll_joint</jointName>
+         		<jointName>	${name}_front_arch_joint, ${name}_back_arch_joint,
+				 			${name}_roll_joint, ${name}_front_roll_joint,
+							${name}_back_roll_joint, ${name}_${chain_name}_1_joint,
+							${name}_${chain_name}_2_joint, ${name}_${chain_name}_3_joint,
+							${name}_${chain_name}_4_joint, ${name}_${chain_name}_5_joint,
+							${name}_${chain_name}_6_joint, ${name}_${chain_name}_7_joint,
+							${name}_${chain_name}_8_joint, ${name}_${chain_name}_9_joint
+				</jointName>
          		<updateRate>10.0</updateRate>
          		<alwaysOn>true</alwaysOn>
        		</plugin>
    		</gazebo>
+		<!-- Foot -->
 		<gazebo reference="${name}_ankle_link">
 			<gravity>true</gravity>
@@ -43,4 +51,41 @@
 			<material>Gazebo/Grey</material>
 		</gazebo>
+		<!-- Chain -->
+		<gazebo reference="${name}_${chain_name}_1_link">
+			<gravity>true</gravity>
+			<material>Gazebo/Grey</material>
+		</gazebo>
+		<gazebo reference="${name}_${chain_name}_2_link">
+			<gravity>true</gravity>
+			<material>Gazebo/Grey</material>
+		</gazebo>
+		<gazebo reference="${name}_${chain_name}_3_link">
+			<gravity>true</gravity>
+			<material>Gazebo/Grey</material>
+		</gazebo>
+		<gazebo reference="${name}_${chain_name}_4_link">
+			<gravity>true</gravity>
+			<material>Gazebo/Grey</material>
+		</gazebo>
+		<gazebo reference="${name}_${chain_name}_5_link">
+			<gravity>true</gravity>
+			<material>Gazebo/Grey</material>
+		</gazebo>
+		<gazebo reference="${name}_${chain_name}_6_link">
+			<gravity>true</gravity>
+			<material>Gazebo/Grey</material>
+		</gazebo>
+		<gazebo reference="${name}_${chain_name}_7_link">
+			<gravity>true</gravity>
+			<material>Gazebo/Grey</material>
+		</gazebo>
+		<gazebo reference="${name}_${chain_name}_8_link">
+			<gravity>true</gravity>
+			<material>Gazebo/Grey</material>
+		</gazebo>
+		<gazebo reference="${name}_${chain_name}_9_link">
+			<gravity>true</gravity>
+			<material>Gazebo/Grey</material>
+		</gazebo>
 	</xacro:macro>
 </robot>

File: softfoot_thing_description/model/softfoot_thing.urdf.xacro (robot description, xacro)
@@ -233,10 +233,10 @@
 		<link name="${name}_back_roll_dummy"/> -->
 		<!-- 5) Chain - joints along y-axis to pitch -->
-		<xacro:chain_thing name="middle_chain" parent="${name}_front_roll_link">
+		<xacro:chain_thing name="middle_chain" foot="${name}" parent="${name}_front_roll_link">
     		<!-- <origin xyz="-0.00209969 0 -0.0118454" rpy="0 0.1046328 0"/> -->
 			<origin xyz="-0.00209969 0 -0.0118454" rpy="${-(const_pi / 2) + 0.1046328} 0 ${const_pi / 2}"/>
   		</xacro:chain_thing>
 		<!-- Gazebo elements -->
-		<xacro:softfoot_thing_gazebo name="${name}"/>
+		<xacro:softfoot_thing_gazebo name="${name}" chain_name="middle_chain"/>
 		<xacro:softfoot_thing_transmission name="${name}"/>
 	</xacro:macro>

Commit message: Now chain revolute axes around x but this needs to be changed

File: softfoot_thing_description/model/chain_thing.urdf.xacro (robot description, xacro)
@@ -12,9 +12,10 @@
 	<!-- URDF -->
 	<xacro:macro name="chain_thing" params="parent name foot *origin">
+		<!-- TODO: Rotation axes now around x, it might be beter to change meshes to revolute around y -->
 		<!-- 0) Chain 1 - joint along y-axis to pitch -->
 		<joint name="${foot}_${name}_1_joint" type="revolute">
 			<xacro:insert_block name="origin"/>
 			<origin xyz="0 0 0" rpy="0 0 0"/>
-			<axis xyz="0 1 0"/>
+			<axis xyz="1 0 0"/>
 			<limit lower="${-45 * const_pi / 180}" upper="${45 * const_pi / 180}" effort="1" velocity="1" />
 			<dynamics friction="0.0001" damping="0.0001"/>
@@ -45,5 +46,5 @@
 		<joint name="${foot}_${name}_2_joint" type="revolute">
 			<origin xyz="0 0 0.0127" rpy="0 0 0"/>
-			<axis xyz="0 1 0"/>
+			<axis xyz="1 0 0"/>
 			<limit lower="${-45 * const_pi / 180}" upper="${45 * const_pi / 180}" effort="1" velocity="1" />
 			<dynamics friction="0.0001" damping="0.0001"/>
@@ -74,5 +75,5 @@
 		<joint name="${foot}_${name}_3_joint" type="revolute">
 			<origin xyz="0 0 0.0127" rpy="0 0 0"/>
-			<axis xyz="0 1 0"/>
+			<axis xyz="1 0 0"/>
 			<limit lower="${-45 * const_pi / 180}" upper="${45 * const_pi / 180}" effort="1" velocity="1" />
 			<dynamics friction="0.0001" damping="0.0001"/>
@@ -103,5 +104,5 @@
 		<joint name="${foot}_${name}_4_joint" type="revolute">
 			<origin xyz="0 0 0.0127" rpy="0 0 0"/>
-			<axis xyz="0 1 0"/>
+			<axis xyz="1 0 0"/>
 			<limit lower="${-45 * const_pi / 180}" upper="${45 * const_pi / 180}" effort="1" velocity="1" />
 			<dynamics friction="0.0001" damping="0.0001"/>
@@ -132,5 +133,5 @@
 		<joint name="${foot}_${name}_5_joint" type="revolute">
 			<origin xyz="0 0 0.0127" rpy="0 0 0"/>
-			<axis xyz="0 1 0"/>
+			<axis xyz="1 0 0"/>
 			<limit lower="${-45 * const_pi / 180}" upper="${45 * const_pi / 180}" effort="1" velocity="1" />
 			<dynamics friction="0.0001" damping="0.0001"/>
@@ -161,5 +162,5 @@
 		<joint name="${foot}_${name}_6_joint" type="revolute">
 			<origin xyz="0 0 0.0127" rpy="0 0 0"/>
-			<axis xyz="0 1 0"/>
+			<axis xyz="1 0 0"/>
 			<limit lower="${-45 * const_pi / 180}" upper="${45 * const_pi / 180}" effort="1" velocity="1" />
 			<dynamics friction="0.0001" damping="0.0001"/>
@@ -190,5 +191,5 @@
 		<joint name="${foot}_${name}_7_joint" type="revolute">
 			<origin xyz="0 0 0.0127" rpy="0 0 0"/>
-			<axis xyz="0 1 0"/>
+			<axis xyz="1 0 0"/>
 			<limit lower="${-45 * const_pi / 180}" upper="${45 * const_pi / 180}" effort="1" velocity="1" />
 			<dynamics friction="0.0001" damping="0.0001"/>
@@ -219,5 +220,5 @@
 		<joint name="${foot}_${name}_8_joint" type="revolute">
 			<origin xyz="0 0 0.0127" rpy="0 0 0"/>
-			<axis xyz="0 1 0"/>
+			<axis xyz="1 0 0"/>
 			<limit lower="${-45 * const_pi / 180}" upper="${45 * const_pi / 180}" effort="1" velocity="1" />
 			<dynamics friction="0.0001" damping="0.0001"/>
@@ -248,5 +249,5 @@
 		<joint name="${foot}_${name}_9_joint" type="revolute">
 			<origin xyz="0 0 0.0127" rpy="0 0 0"/>
-			<axis xyz="0 1 0"/>
+			<axis xyz="1 0 0"/>
 			<limit lower="${-45 * const_pi / 180}" upper="${45 * const_pi / 180}" effort="1" velocity="1" />
 			<dynamics friction="0.0001" damping="0.0001"/>

Commit message: Added links for chain ik reconstruction

File: softfoot_thing_description/model/chain_thing.urdf.xacro (robot description, xacro)
@@ -275,4 +275,11 @@
 			</collision>
 		</link>
+		<!-- 9) Chain Tip - fixed joint -->
+		<joint name="${foot}_${name}_tip_joint" type="fixed">
+			<origin xyz="0 0 0.0127" rpy="0 0 0"/>
+			<parent link="${foot}_${name}_9_link"/>
+			<child link="${foot}_${name}_tip_link"/>
+		</joint>
+		<link name="${foot}_${name}_tip_link"/>
 	</xacro:macro>
 </robot>

File: softfoot_thing_description/model/softfoot_thing.urdf.xacro (robot description, xacro)
@@ -232,7 +232,13 @@
 		</joint>
 		<link name="${name}_back_roll_dummy"/> -->
-		<!-- 5) Chain - joints along y-axis to pitch -->
+		<!-- 5) Chain insertion point -->
+        <joint name="${name}_chain_insertion_joint" type="fixed">
+			<origin xyz="-0.00209969 0 -0.0118454" rpy="${-(const_pi / 2) - 0.105} 0 ${-const_pi / 2}"/>
+			<parent link="${name}_back_roll_link"/>
+			<child link="${name}_chain_insertion_link"/>
+		</joint>
+		<link name="${name}_chain_insertion_link"/>
+		<!-- 6) Chain - starting from front -->
 		<xacro:chain_thing name="middle_chain" foot="${name}" parent="${name}_front_roll_link">
-    		<!-- <origin xyz="-0.00209969 0 -0.0118454" rpy="0 0.1046328 0"/> -->
 			<origin xyz="-0.00209969 0 -0.0118454" rpy="${-(const_pi / 2) + 0.1046328} 0 ${const_pi / 2}"/>
   		</xacro:chain_thing>

Commit message: Playing with values to inrease simulation precision

File: softfoot_thing_description/model/chain_thing.urdf.xacro (robot description, xacro)
@@ -12,5 +12,5 @@
 	<!-- URDF -->
 	<xacro:macro name="chain_thing" params="parent name foot *origin">
-		<!-- TODO: Rotation axes now around x, it might be beter to change meshes to revolute around y -->
+		<!-- TODO: Rotation axes now around x, it might be better to change meshes to revolute around y -->
 		<!-- 0) Chain 1 - joint along y-axis to pitch -->
 		<joint name="${foot}_${name}_1_joint" type="revolute">
@@ -18,5 +18,5 @@
 			<origin xyz="0 0 0" rpy="0 0 0"/>
 			<axis xyz="1 0 0"/>
-			<limit lower="${-45 * const_pi / 180}" upper="${45 * const_pi / 180}" effort="1" velocity="1" />
+			<limit lower="${0 * const_pi / 180}" upper="${45 * const_pi / 180}" effort="1" velocity="1" />
 			<dynamics friction="0.0001" damping="0.0001"/>
 			<parent link="${parent}"/>
@@ -47,5 +47,5 @@
 			<origin xyz="0 0 0.0127" rpy="0 0 0"/>
 			<axis xyz="1 0 0"/>
-			<limit lower="${-45 * const_pi / 180}" upper="${45 * const_pi / 180}" effort="1" velocity="1" />
+			<limit lower="${-5 * const_pi / 180}" upper="${45 * const_pi / 180}" effort="1" velocity="1" />
 			<dynamics friction="0.0001" damping="0.0001"/>
 			<parent link="${foot}_${name}_1_link"/>
@@ -76,5 +76,5 @@
 			<origin xyz="0 0 0.0127" rpy="0 0 0"/>
 			<axis xyz="1 0 0"/>
-			<limit lower="${-45 * const_pi / 180}" upper="${45 * const_pi / 180}" effort="1" velocity="1" />
+			<limit lower="${-10 * const_pi / 180}" upper="${45 * const_pi / 180}" effort="1" velocity="1" />
 			<dynamics friction="0.0001" damping="0.0001"/>
 			<parent link="${foot}_${name}_2_link"/>
@@ -105,5 +105,5 @@
 			<origin xyz="0 0 0.0127" rpy="0 0 0"/>
 			<axis xyz="1 0 0"/>
-			<limit lower="${-45 * const_pi / 180}" upper="${45 * const_pi / 180}" effort="1" velocity="1" />
+			<limit lower="${-15 * const_pi / 180}" upper="${45 * const_pi / 180}" effort="1" velocity="1" />
 			<dynamics friction="0.0001" damping="0.0001"/>
 			<parent link="${foot}_${name}_3_link"/>
@@ -134,5 +134,5 @@
 			<origin xyz="0 0 0.0127" rpy="0 0 0"/>
 			<axis xyz="1 0 0"/>
-			<limit lower="${-45 * const_pi / 180}" upper="${45 * const_pi / 180}" effort="1" velocity="1" />
+			<limit lower="${-20 * const_pi / 180}" upper="${45 * const_pi / 180}" effort="1" velocity="1" />
 			<dynamics friction="0.0001" damping="0.0001"/>
 			<parent link="${foot}_${name}_4_link"/>
@@ -163,5 +163,5 @@
 			<origin xyz="0 0 0.0127" rpy="0 0 0"/>
 			<axis xyz="1 0 0"/>
-			<limit lower="${-45 * const_pi / 180}" upper="${45 * const_pi / 180}" effort="1" velocity="1" />
+			<limit lower="${-25 * const_pi / 180}" upper="${45 * const_pi / 180}" effort="1" velocity="1" />
 			<dynamics friction="0.0001" damping="0.0001"/>
 			<parent link="${foot}_${name}_5_link"/>
@@ -192,5 +192,5 @@
 			<origin xyz="0 0 0.0127" rpy="0 0 0"/>
 			<axis xyz="1 0 0"/>
-			<limit lower="${-45 * const_pi / 180}" upper="${45 * const_pi / 180}" effort="1" velocity="1" />
+			<limit lower="${-30 * const_pi / 180}" upper="${45 * const_pi / 180}" effort="1" velocity="1" />
 			<dynamics friction="0.0001" damping="0.0001"/>
 			<parent link="${foot}_${name}_6_link"/>
@@ -221,5 +221,5 @@
 			<origin xyz="0 0 0.0127" rpy="0 0 0"/>
 			<axis xyz="1 0 0"/>
-			<limit lower="${-45 * const_pi / 180}" upper="${45 * const_pi / 180}" effort="1" velocity="1" />
+			<limit lower="${-35 * const_pi / 180}" upper="${45 * const_pi / 180}" effort="1" velocity="1" />
 			<dynamics friction="0.0001" damping="0.0001"/>
 			<parent link="${foot}_${name}_7_link"/>
@@ -250,5 +250,5 @@
 			<origin xyz="0 0 0.0127" rpy="0 0 0"/>
 			<axis xyz="1 0 0"/>
-			<limit lower="${-45 * const_pi / 180}" upper="${45 * const_pi / 180}" effort="1" velocity="1" />
+			<limit lower="${-40 * const_pi / 180}" upper="${45 * const_pi / 180}" effort="1" velocity="1" />
 			<dynamics friction="0.0001" damping="0.0001"/>
 			<parent link="${foot}_${name}_8_link"/>
