Commit message: Modified limits and fixed base guess is always used to compute ik

File: softfoot_thing_description/model/chain_thing.urdf.xacro (robot description, xacro)
@@ -18,5 +18,5 @@
 			<origin xyz="0 0 0" rpy="0 0 0"/>
 			<axis xyz="1 0 0"/>
-			<limit lower="${0 * const_pi / 180}" upper="${45 * const_pi / 180}" effort="1" velocity="1" />
+			<limit lower="${0 * const_pi / 180}" upper="${40 * const_pi / 180}" effort="1" velocity="1" />
 			<dynamics friction="0.0001" damping="0.0001"/>
 			<parent link="${parent}"/>
@@ -47,5 +47,5 @@
 			<origin xyz="0 0 0.0127" rpy="0 0 0"/>
 			<axis xyz="1 0 0"/>
-			<limit lower="${-5 * const_pi / 180}" upper="${45 * const_pi / 180}" effort="1" velocity="1" />
+			<limit lower="${-5 * const_pi / 180}" upper="${35 * const_pi / 180}" effort="1" velocity="1" />
 			<dynamics friction="0.0001" damping="0.0001"/>
 			<parent link="${foot}_${name}_1_link"/>
@@ -76,5 +76,5 @@
 			<origin xyz="0 0 0.0127" rpy="0 0 0"/>
 			<axis xyz="1 0 0"/>
-			<limit lower="${-10 * const_pi / 180}" upper="${45 * const_pi / 180}" effort="1" velocity="1" />
+			<limit lower="${-10 * const_pi / 180}" upper="${30 * const_pi / 180}" effort="1" velocity="1" />
 			<dynamics friction="0.0001" damping="0.0001"/>
 			<parent link="${foot}_${name}_2_link"/>
@@ -105,5 +105,5 @@
 			<origin xyz="0 0 0.0127" rpy="0 0 0"/>
 			<axis xyz="1 0 0"/>
-			<limit lower="${-15 * const_pi / 180}" upper="${45 * const_pi / 180}" effort="1" velocity="1" />
+			<limit lower="${-15 * const_pi / 180}" upper="${25 * const_pi / 180}" effort="1" velocity="1" />
 			<dynamics friction="0.0001" damping="0.0001"/>
 			<parent link="${foot}_${name}_3_link"/>
@@ -134,5 +134,5 @@
 			<origin xyz="0 0 0.0127" rpy="0 0 0"/>
 			<axis xyz="1 0 0"/>
-			<limit lower="${-20 * const_pi / 180}" upper="${45 * const_pi / 180}" effort="1" velocity="1" />
+			<limit lower="${-20 * const_pi / 180}" upper="${20 * const_pi / 180}" effort="1" velocity="1" />
 			<dynamics friction="0.0001" damping="0.0001"/>
 			<parent link="${foot}_${name}_4_link"/>
@@ -163,5 +163,5 @@
 			<origin xyz="0 0 0.0127" rpy="0 0 0"/>
 			<axis xyz="1 0 0"/>
-			<limit lower="${-25 * const_pi / 180}" upper="${45 * const_pi / 180}" effort="1" velocity="1" />
+			<limit lower="${-25 * const_pi / 180}" upper="${15 * const_pi / 180}" effort="1" velocity="1" />
 			<dynamics friction="0.0001" damping="0.0001"/>
 			<parent link="${foot}_${name}_5_link"/>
@@ -192,5 +192,5 @@
 			<origin xyz="0 0 0.0127" rpy="0 0 0"/>
 			<axis xyz="1 0 0"/>
-			<limit lower="${-30 * const_pi / 180}" upper="${45 * const_pi / 180}" effort="1" velocity="1" />
+			<limit lower="${-30 * const_pi / 180}" upper="${10 * const_pi / 180}" effort="1" velocity="1" />
 			<dynamics friction="0.0001" damping="0.0001"/>
 			<parent link="${foot}_${name}_6_link"/>
@@ -221,5 +221,5 @@
 			<origin xyz="0 0 0.0127" rpy="0 0 0"/>
 			<axis xyz="1 0 0"/>
-			<limit lower="${-35 * const_pi / 180}" upper="${45 * const_pi / 180}" effort="1" velocity="1" />
+			<limit lower="${-35 * const_pi / 180}" upper="${5 * const_pi / 180}" effort="1" velocity="1" />
 			<dynamics friction="0.0001" damping="0.0001"/>
 			<parent link="${foot}_${name}_7_link"/>
@@ -250,5 +250,5 @@
 			<origin xyz="0 0 0.0127" rpy="0 0 0"/>
 			<axis xyz="1 0 0"/>
-			<limit lower="${-40 * const_pi / 180}" upper="${45 * const_pi / 180}" effort="1" velocity="1" />
+			<limit lower="${-40 * const_pi / 180}" upper="${0 * const_pi / 180}" effort="1" velocity="1" />
 			<dynamics friction="0.0001" damping="0.0001"/>
 			<parent link="${foot}_${name}_8_link"/>

Commit message: Restored natural limits on chain joints

File: softfoot_thing_description/model/chain_thing.urdf.xacro (robot description, xacro)
@@ -18,5 +18,5 @@
 			<origin xyz="0 0 0" rpy="0 0 0"/>
 			<axis xyz="1 0 0"/>
-			<limit lower="${0 * const_pi / 180}" upper="${40 * const_pi / 180}" effort="1" velocity="1" />
+			<limit lower="${-45 * const_pi / 180}" upper="${45 * const_pi / 180}" effort="1" velocity="1" />
 			<dynamics friction="0.0001" damping="0.0001"/>
 			<parent link="${parent}"/>
@@ -47,5 +47,5 @@
 			<origin xyz="0 0 0.0127" rpy="0 0 0"/>
 			<axis xyz="1 0 0"/>
-			<limit lower="${-5 * const_pi / 180}" upper="${35 * const_pi / 180}" effort="1" velocity="1" />
+			<limit lower="${-45 * const_pi / 180}" upper="${45 * const_pi / 180}" effort="1" velocity="1" />
 			<dynamics friction="0.0001" damping="0.0001"/>
 			<parent link="${foot}_${name}_1_link"/>
@@ -76,5 +76,5 @@
 			<origin xyz="0 0 0.0127" rpy="0 0 0"/>
 			<axis xyz="1 0 0"/>
-			<limit lower="${-10 * const_pi / 180}" upper="${30 * const_pi / 180}" effort="1" velocity="1" />
+			<limit lower="${-45 * const_pi / 180}" upper="${45 * const_pi / 180}" effort="1" velocity="1" />
 			<dynamics friction="0.0001" damping="0.0001"/>
 			<parent link="${foot}_${name}_2_link"/>
@@ -105,5 +105,5 @@
 			<origin xyz="0 0 0.0127" rpy="0 0 0"/>
 			<axis xyz="1 0 0"/>
-			<limit lower="${-15 * const_pi / 180}" upper="${25 * const_pi / 180}" effort="1" velocity="1" />
+			<limit lower="${-45 * const_pi / 180}" upper="${45 * const_pi / 180}" effort="1" velocity="1" />
 			<dynamics friction="0.0001" damping="0.0001"/>
 			<parent link="${foot}_${name}_3_link"/>
@@ -134,5 +134,5 @@
 			<origin xyz="0 0 0.0127" rpy="0 0 0"/>
 			<axis xyz="1 0 0"/>
-			<limit lower="${-20 * const_pi / 180}" upper="${20 * const_pi / 180}" effort="1" velocity="1" />
+			<limit lower="${-45 * const_pi / 180}" upper="${45 * const_pi / 180}" effort="1" velocity="1" />
 			<dynamics friction="0.0001" damping="0.0001"/>
 			<parent link="${foot}_${name}_4_link"/>
@@ -163,5 +163,5 @@
 			<origin xyz="0 0 0.0127" rpy="0 0 0"/>
 			<axis xyz="1 0 0"/>
-			<limit lower="${-25 * const_pi / 180}" upper="${15 * const_pi / 180}" effort="1" velocity="1" />
+			<limit lower="${-45 * const_pi / 180}" upper="${45 * const_pi / 180}" effort="1" velocity="1" />
 			<dynamics friction="0.0001" damping="0.0001"/>
 			<parent link="${foot}_${name}_5_link"/>
@@ -192,5 +192,5 @@
 			<origin xyz="0 0 0.0127" rpy="0 0 0"/>
 			<axis xyz="1 0 0"/>
-			<limit lower="${-30 * const_pi / 180}" upper="${10 * const_pi / 180}" effort="1" velocity="1" />
+			<limit lower="${-45 * const_pi / 180}" upper="${45 * const_pi / 180}" effort="1" velocity="1" />
 			<dynamics friction="0.0001" damping="0.0001"/>
 			<parent link="${foot}_${name}_6_link"/>
@@ -221,5 +221,5 @@
 			<origin xyz="0 0 0.0127" rpy="0 0 0"/>
 			<axis xyz="1 0 0"/>
-			<limit lower="${-35 * const_pi / 180}" upper="${5 * const_pi / 180}" effort="1" velocity="1" />
+			<limit lower="${-45 * const_pi / 180}" upper="${45 * const_pi / 180}" effort="1" velocity="1" />
 			<dynamics friction="0.0001" damping="0.0001"/>
 			<parent link="${foot}_${name}_7_link"/>
@@ -250,5 +250,5 @@
 			<origin xyz="0 0 0.0127" rpy="0 0 0"/>
 			<axis xyz="1 0 0"/>
-			<limit lower="${-40 * const_pi / 180}" upper="${0 * const_pi / 180}" effort="1" velocity="1" />
+			<limit lower="${-45 * const_pi / 180}" upper="${45 * const_pi / 180}" effort="1" velocity="1" />
 			<dynamics friction="0.0001" damping="0.0001"/>
 			<parent link="${foot}_${name}_8_link"/>

Commit message: Modifications for gazebo plugin

File: softfoot_thing_description/model/chain_thing.urdf.xacro (robot description, xacro)
@@ -281,5 +281,6 @@
 			<child link="${foot}_${name}_tip_link"/>
 		</joint>
-		<link name="${foot}_${name}_tip_link"/>
+                <link name="${foot}_${name}_tip_link">
+                </link>
 	</xacro:macro>
 </robot>

File: softfoot_thing_description/model/softfoot_thing.gazebo.xacro (robot description, xacro)
@@ -19,11 +19,11 @@
          		<robotNamespace>${name}</robotNamespace>
          		<jointName>	${name}_front_arch_joint, ${name}_back_arch_joint,
-				 			${name}_roll_joint, ${name}_front_roll_joint,
-							${name}_back_roll_joint, ${name}_${chain_name}_1_joint,
-							${name}_${chain_name}_2_joint, ${name}_${chain_name}_3_joint,
-							${name}_${chain_name}_4_joint, ${name}_${chain_name}_5_joint,
-							${name}_${chain_name}_6_joint, ${name}_${chain_name}_7_joint,
-							${name}_${chain_name}_8_joint, ${name}_${chain_name}_9_joint
-				</jointName>
+                                        ${name}_roll_joint, ${name}_front_roll_joint,
+                                        ${name}_back_roll_joint, ${name}_${chain_name}_1_joint,
+                                        ${name}_${chain_name}_2_joint, ${name}_${chain_name}_3_joint,
+                                        ${name}_${chain_name}_4_joint, ${name}_${chain_name}_5_joint,
+                                        ${name}_${chain_name}_6_joint, ${name}_${chain_name}_7_joint,
+                                        ${name}_${chain_name}_8_joint, ${name}_${chain_name}_9_joint
+                        </jointName>
          		<updateRate>10.0</updateRate>
          		<alwaysOn>true</alwaysOn>
@@ -56,4 +56,9 @@
 			<material>Gazebo/Grey</material>
 		</gazebo>
+                <gazebo reference="${name}_${chain_name}_insertion_link">
+                        <gravity>true</gravity>
+                        <!--<selfCollide>true</selfCollide>-->
+                        <material>Gazebo/Grey</material>
+                </gazebo>
 		<!-- Chain -->
 		<gazebo reference="${name}_${chain_name}_1_link">
@@ -102,4 +107,9 @@
 			<material>Gazebo/Grey</material>
 		</gazebo>
+                <gazebo reference="${name}_${chain_name}_tip_link">
+                        <gravity>true</gravity>
+                        <!-- <selfCollide>true</selfCollide> -->
+                        <material>Gazebo/Grey</material>
+                </gazebo>
 	</xacro:macro>
 </robot>

File: softfoot_thing_description/robot/pisa_softfoot.urdf.xacro (robot description, xacro)
@@ -1,49 +1,49 @@
 <?xml version="1.0" encoding='utf-8'?>
 <robot xmlns:xacro="http://www.ros.org/wiki/xacro" name="pisa_softfoot">
-  <!-- ARGS -->
-  <xacro:property name="leg_mass" value="0.02"/>
-  <!-- MODELS -->
-  <xacro:include filename="$(find softfoot_thing_description)/model/softfoot_thing.urdf.xacro"/>
-  <!-- WORLD -->
-  <link name="world">
-  </link>
-  <!-- LEG 1 -->
-  <joint name="world_to_leg_3" type="revolute">
+<!-- ARGS -->
+<xacro:property name="leg_mass" value="0.02"/>
+<!-- MODELS -->
+<xacro:include filename="$(find softfoot_thing_description)/model/softfoot_thing.urdf.xacro"/>
+<!-- WORLD -->
+<link name="world">
+</link>
+<!-- LEG 1 -->
+<joint name="world_to_leg_3" type="revolute">
     <origin xyz="0 0 0.2" rpy="0 0 0"/>
     <axis xyz="0 1 0"/>
     <limit lower="-0.50" upper="0.50" effort="1" velocity="1" />
-		<dynamics friction="0.01" damping="0.01"/>
+    <dynamics friction="0.01" damping="0.01"/>
     <parent link="world"/>
     <child link="leg_link_3"/>
-  </joint>
-  <link name="leg_link_3">
+</joint>
+<link name="leg_link_3">
     <inertial>
-			<mass value="${leg_mass}"/>
-			<origin xyz="0 0 0" rpy="0 0 0"/>
-			<inertia  ixx="${mm2tom2 * 1}" iyy="${mm2tom2 * 1}" izz="${mm2tom2 * 1}"
-                ixy="0" ixz="0" iyz="0"/>
-		</inertial>
+        <mass value="${leg_mass}"/>
+        <origin xyz="0 0 0" rpy="0 0 0"/>
+        <inertia    ixx="${mm2tom2 * 1}" iyy="${mm2tom2 * 1}" izz="${mm2tom2 * 1}"
+                    ixy="0" ixz="0" iyz="0"/>
+        </inertial>
     <visual>
-      <origin xyz="0 0 0" rpy="0 0 0"/>
-      <geometry>
-        <cylinder length="0.1" radius="0.015"/>
-      </geometry>
-      <material name="SoftFoot/Black"/>
+        <origin xyz="0 0 0" rpy="0 0 0"/>
+        <geometry>
+            <cylinder length="0.1" radius="0.015"/>
+        </geometry>
+        <material name="SoftFoot/Black"/>
     </visual>
     <collision>
-			<origin xyz="0 0 0" rpy="0 0 0"/>
-			<geometry>
-        <cylinder length="0.1" radius="0.015"/>
-      </geometry>
-		</collision>
-  </link>
-  <gazebo reference="leg_link_3">
-		<gravity>true</gravity>
-		<material>Gazebo/Black</material>
-	</gazebo>
-  <!-- FOOT 1 -->
-  <xacro:softfoot_thing name="softfoot_3" parent="leg_link_3">
+        <origin xyz="0 0 0" rpy="0 0 0"/>
+        <geometry>
+            <cylinder length="0.1" radius="0.015"/>
+        </geometry>
+    </collision>
+</link>
+<gazebo reference="leg_link_3">
+    <gravity>true</gravity>
+    <material>Gazebo/Black</material>
+</gazebo>
+<!-- FOOT 1 -->
+<xacro:softfoot_thing name="softfoot_3" parent="leg_link_3">
     <origin xyz="0 0 -0.05" rpy="0 0 0"/>
-  </xacro:softfoot_thing>
+</xacro:softfoot_thing>
   <!-- LEG 2 -->
   <!-- <joint name="world_to_leg_4" type="fixed">

Commit message: More realistic limits for chain

File: softfoot_thing_description/model/chain_thing.urdf.xacro (robot description, xacro)
@@ -18,5 +18,5 @@
 			<origin xyz="0 0 0" rpy="0 0 0"/>
 			<axis xyz="1 0 0"/>
-			<limit lower="${-45 * const_pi / 180}" upper="${45 * const_pi / 180}" effort="1" velocity="1" />
+                        <limit lower="${-15 * const_pi / 180}" upper="${15 * const_pi / 180}" effort="1" velocity="1" />
 			<dynamics friction="0.0001" damping="0.0001"/>
 			<parent link="${parent}"/>
@@ -47,5 +47,5 @@
 			<origin xyz="0 0 0.0127" rpy="0 0 0"/>
 			<axis xyz="1 0 0"/>
-			<limit lower="${-45 * const_pi / 180}" upper="${45 * const_pi / 180}" effort="1" velocity="1" />
+                        <limit lower="${-15 * const_pi / 180}" upper="${15 * const_pi / 180}" effort="1" velocity="1" />
 			<dynamics friction="0.0001" damping="0.0001"/>
 			<parent link="${foot}_${name}_1_link"/>
@@ -76,5 +76,5 @@
 			<origin xyz="0 0 0.0127" rpy="0 0 0"/>
 			<axis xyz="1 0 0"/>
-			<limit lower="${-45 * const_pi / 180}" upper="${45 * const_pi / 180}" effort="1" velocity="1" />
+                        <limit lower="${-15 * const_pi / 180}" upper="${15 * const_pi / 180}" effort="1" velocity="1" />
 			<dynamics friction="0.0001" damping="0.0001"/>
 			<parent link="${foot}_${name}_2_link"/>
@@ -105,5 +105,5 @@
 			<origin xyz="0 0 0.0127" rpy="0 0 0"/>
 			<axis xyz="1 0 0"/>
-			<limit lower="${-45 * const_pi / 180}" upper="${45 * const_pi / 180}" effort="1" velocity="1" />
+                        <limit lower="${-15 * const_pi / 180}" upper="${15 * const_pi / 180}" effort="1" velocity="1" />
 			<dynamics friction="0.0001" damping="0.0001"/>
 			<parent link="${foot}_${name}_3_link"/>
@@ -134,5 +134,5 @@
 			<origin xyz="0 0 0.0127" rpy="0 0 0"/>
 			<axis xyz="1 0 0"/>
-			<limit lower="${-45 * const_pi / 180}" upper="${45 * const_pi / 180}" effort="1" velocity="1" />
+                        <limit lower="${-15 * const_pi / 180}" upper="${15 * const_pi / 180}" effort="1" velocity="1" />
 			<dynamics friction="0.0001" damping="0.0001"/>
 			<parent link="${foot}_${name}_4_link"/>
@@ -163,5 +163,5 @@
 			<origin xyz="0 0 0.0127" rpy="0 0 0"/>
 			<axis xyz="1 0 0"/>
-			<limit lower="${-45 * const_pi / 180}" upper="${45 * const_pi / 180}" effort="1" velocity="1" />
+                        <limit lower="${-15 * const_pi / 180}" upper="${15 * const_pi / 180}" effort="1" velocity="1" />
 			<dynamics friction="0.0001" damping="0.0001"/>
 			<parent link="${foot}_${name}_5_link"/>
@@ -192,5 +192,5 @@
 			<origin xyz="0 0 0.0127" rpy="0 0 0"/>
 			<axis xyz="1 0 0"/>
-			<limit lower="${-45 * const_pi / 180}" upper="${45 * const_pi / 180}" effort="1" velocity="1" />
+                        <limit lower="${-15 * const_pi / 180}" upper="${15 * const_pi / 180}" effort="1" velocity="1" />
 			<dynamics friction="0.0001" damping="0.0001"/>
 			<parent link="${foot}_${name}_6_link"/>
@@ -221,5 +221,5 @@
 			<origin xyz="0 0 0.0127" rpy="0 0 0"/>
 			<axis xyz="1 0 0"/>
-			<limit lower="${-45 * const_pi / 180}" upper="${45 * const_pi / 180}" effort="1" velocity="1" />
+                        <limit lower="${-15 * const_pi / 180}" upper="${15 * const_pi / 180}" effort="1" velocity="1" />
 			<dynamics friction="0.0001" damping="0.0001"/>
 			<parent link="${foot}_${name}_7_link"/>
@@ -250,5 +250,5 @@
 			<origin xyz="0 0 0.0127" rpy="0 0 0"/>
 			<axis xyz="1 0 0"/>
-			<limit lower="${-45 * const_pi / 180}" upper="${45 * const_pi / 180}" effort="1" velocity="1" />
+                        <limit lower="${-15 * const_pi / 180}" upper="${15 * const_pi / 180}" effort="1" velocity="1" />
 			<dynamics friction="0.0001" damping="0.0001"/>
 			<parent link="${foot}_${name}_8_link"/>

Commit message: Restored actual chain joint limits

File: softfoot_thing_description/model/chain_thing.urdf.xacro (robot description, xacro)
@@ -18,5 +18,5 @@
 			<origin xyz="0 0 0" rpy="0 0 0"/>
 			<axis xyz="1 0 0"/>
-                        <limit lower="${-15 * const_pi / 180}" upper="${15 * const_pi / 180}" effort="1" velocity="1" />
+                        <limit lower="${-45 * const_pi / 180}" upper="${45 * const_pi / 180}" effort="1" velocity="1" />
 			<dynamics friction="0.0001" damping="0.0001"/>
 			<parent link="${parent}"/>
@@ -47,5 +47,5 @@
 			<origin xyz="0 0 0.0127" rpy="0 0 0"/>
 			<axis xyz="1 0 0"/>
-                        <limit lower="${-15 * const_pi / 180}" upper="${15 * const_pi / 180}" effort="1" velocity="1" />
+                        <limit lower="${-45 * const_pi / 180}" upper="${45 * const_pi / 180}" effort="1" velocity="1" />
 			<dynamics friction="0.0001" damping="0.0001"/>
 			<parent link="${foot}_${name}_1_link"/>
@@ -76,5 +76,5 @@
 			<origin xyz="0 0 0.0127" rpy="0 0 0"/>
 			<axis xyz="1 0 0"/>
-                        <limit lower="${-15 * const_pi / 180}" upper="${15 * const_pi / 180}" effort="1" velocity="1" />
+                        <limit lower="${-45 * const_pi / 180}" upper="${45 * const_pi / 180}" effort="1" velocity="1" />
 			<dynamics friction="0.0001" damping="0.0001"/>
 			<parent link="${foot}_${name}_2_link"/>
@@ -105,5 +105,5 @@
 			<origin xyz="0 0 0.0127" rpy="0 0 0"/>
 			<axis xyz="1 0 0"/>
-                        <limit lower="${-15 * const_pi / 180}" upper="${15 * const_pi / 180}" effort="1" velocity="1" />
+                        <limit lower="${-45 * const_pi / 180}" upper="${45 * const_pi / 180}" effort="1" velocity="1" />
 			<dynamics friction="0.0001" damping="0.0001"/>
 			<parent link="${foot}_${name}_3_link"/>
@@ -134,5 +134,5 @@
 			<origin xyz="0 0 0.0127" rpy="0 0 0"/>
 			<axis xyz="1 0 0"/>
-                        <limit lower="${-15 * const_pi / 180}" upper="${15 * const_pi / 180}" effort="1" velocity="1" />
+                        <limit lower="${-45 * const_pi / 180}" upper="${45 * const_pi / 180}" effort="1" velocity="1" />
 			<dynamics friction="0.0001" damping="0.0001"/>
 			<parent link="${foot}_${name}_4_link"/>
@@ -163,5 +163,5 @@
 			<origin xyz="0 0 0.0127" rpy="0 0 0"/>
 			<axis xyz="1 0 0"/>
-                        <limit lower="${-15 * const_pi / 180}" upper="${15 * const_pi / 180}" effort="1" velocity="1" />
+                        <limit lower="${-45 * const_pi / 180}" upper="${45 * const_pi / 180}" effort="1" velocity="1" />
 			<dynamics friction="0.0001" damping="0.0001"/>
 			<parent link="${foot}_${name}_5_link"/>
@@ -192,5 +192,5 @@
 			<origin xyz="0 0 0.0127" rpy="0 0 0"/>
 			<axis xyz="1 0 0"/>
-                        <limit lower="${-15 * const_pi / 180}" upper="${15 * const_pi / 180}" effort="1" velocity="1" />
+                        <limit lower="${-45 * const_pi / 180}" upper="${45 * const_pi / 180}" effort="1" velocity="1" />
 			<dynamics friction="0.0001" damping="0.0001"/>
 			<parent link="${foot}_${name}_6_link"/>
@@ -221,5 +221,5 @@
 			<origin xyz="0 0 0.0127" rpy="0 0 0"/>
 			<axis xyz="1 0 0"/>
-                        <limit lower="${-15 * const_pi / 180}" upper="${15 * const_pi / 180}" effort="1" velocity="1" />
+                        <limit lower="${-45 * const_pi / 180}" upper="${45 * const_pi / 180}" effort="1" velocity="1" />
 			<dynamics friction="0.0001" damping="0.0001"/>
 			<parent link="${foot}_${name}_7_link"/>
@@ -250,5 +250,5 @@
 			<origin xyz="0 0 0.0127" rpy="0 0 0"/>
 			<axis xyz="1 0 0"/>
-                        <limit lower="${-15 * const_pi / 180}" upper="${15 * const_pi / 180}" effort="1" velocity="1" />
+                        <limit lower="${-45 * const_pi / 180}" upper="${45 * const_pi / 180}" effort="1" velocity="1" />
 			<dynamics friction="0.0001" damping="0.0001"/>
 			<parent link="${foot}_${name}_8_link"/>
