Commit message: Tuned mesh quality quality/speed trade-off

File: softfoot_thing_description/model/chain_thing.urdf.xacro (robot description, xacro)
@@ -39,5 +39,5 @@
 				<origin xyz="0 0 0" rpy="0 0 0"/>
 				<geometry>
-					<mesh filename="package://softfoot_thing_description/meshes/visual/inner_chain.stl" scale=" .001 .001 .001"/>
+                                        <mesh filename="package://softfoot_thing_description/meshes/collision/inner_chain.stl" scale=" .001 .001 .001"/>
 				</geometry>
 			</collision>
@@ -68,5 +68,5 @@
 				<origin xyz="0 0 0" rpy="0 0 0"/>
 				<geometry>
-					<mesh filename="package://softfoot_thing_description/meshes/visual/outer_chain.stl" scale=" .001 .001 .001"/>
+                                        <mesh filename="package://softfoot_thing_description/meshes/collision/outer_chain.stl" scale=" .001 .001 .001"/>
 				</geometry>
 			</collision>
@@ -97,5 +97,5 @@
 				<origin xyz="0 0 0" rpy="0 0 0"/>
 				<geometry>
-					<mesh filename="package://softfoot_thing_description/meshes/visual/inner_chain.stl" scale=" .001 .001 .001"/>
+                                        <mesh filename="package://softfoot_thing_description/meshes/collision/inner_chain.stl" scale=" .001 .001 .001"/>
 				</geometry>
 			</collision>
@@ -126,5 +126,5 @@
 				<origin xyz="0 0 0" rpy="0 0 0"/>
 				<geometry>
-					<mesh filename="package://softfoot_thing_description/meshes/visual/outer_chain.stl" scale=" .001 .001 .001"/>
+                                        <mesh filename="package://softfoot_thing_description/meshes/collision/outer_chain.stl" scale=" .001 .001 .001"/>
 				</geometry>
 			</collision>
@@ -155,5 +155,5 @@
 				<origin xyz="0 0 0" rpy="0 0 0"/>
 				<geometry>
-					<mesh filename="package://softfoot_thing_description/meshes/visual/inner_chain.stl" scale=" .001 .001 .001"/>
+                                        <mesh filename="package://softfoot_thing_description/meshes/collision/inner_chain.stl" scale=" .001 .001 .001"/>
 				</geometry>
 			</collision>
@@ -184,5 +184,5 @@
 				<origin xyz="0 0 0" rpy="0 0 0"/>
 				<geometry>
-					<mesh filename="package://softfoot_thing_description/meshes/visual/outer_chain.stl" scale=" .001 .001 .001"/>
+                                        <mesh filename="package://softfoot_thing_description/meshes/collision/outer_chain.stl" scale=" .001 .001 .001"/>
 				</geometry>
 			</collision>
@@ -213,5 +213,5 @@
 				<origin xyz="0 0 0" rpy="0 0 0"/>
 				<geometry>
-					<mesh filename="package://softfoot_thing_description/meshes/visual/inner_chain.stl" scale=" .001 .001 .001"/>
+                                        <mesh filename="package://softfoot_thing_description/meshes/collision/inner_chain.stl" scale=" .001 .001 .001"/>
 				</geometry>
 			</collision>
@@ -242,5 +242,5 @@
 				<origin xyz="0 0 0" rpy="0 0 0"/>
 				<geometry>
-					<mesh filename="package://softfoot_thing_description/meshes/visual/outer_chain.stl" scale=" .001 .001 .001"/>
+                                        <mesh filename="package://softfoot_thing_description/meshes/collision/outer_chain.stl" scale=" .001 .001 .001"/>
 				</geometry>
 			</collision>
@@ -271,5 +271,5 @@
 				<origin xyz="0 0 0" rpy="0 0 0"/>
 				<geometry>
-					<mesh filename="package://softfoot_thing_description/meshes/visual/inner_chain.stl" scale=" .001 .001 .001"/>
+                                        <mesh filename="package://softfoot_thing_description/meshes/collision/inner_chain.stl" scale=" .001 .001 .001"/>
 				</geometry>
 			</collision>

File: softfoot_thing_description/model/softfoot_thing.urdf.xacro (robot description, xacro)
@@ -54,5 +54,5 @@
 				<origin xyz="0 0 0" rpy="0 0 0"/>
 				<geometry>
-					<mesh filename="package://softfoot_thing_description/meshes/visual/ankle.stl" scale=" .001 .001 .001"/>
+                                        <mesh filename="package://softfoot_thing_description/meshes/collision/ankle.stl" scale=" .001 .001 .001"/>
 				</geometry>
 			</collision>
@@ -83,5 +83,5 @@
 				<origin xyz="0 0 0" rpy="0 0 0"/>
 				<geometry>
-					<mesh filename="package://softfoot_thing_description/meshes/visual/front_arch_front.stl" scale=" .001 .001 .001"/>
+                                        <mesh filename="package://softfoot_thing_description/meshes/collision/front_arch_front.stl" scale=" .001 .001 .001"/>
 				</geometry>
 			</collision>
@@ -122,5 +122,5 @@
 				<origin xyz="0 0 0" rpy="0 0 0"/>
 				<geometry>
-					<mesh filename="package://softfoot_thing_description/meshes/visual/front_arch_back.stl" scale=" .001 .001 .001"/>
+                                        <mesh filename="package://softfoot_thing_description/meshes/collision/front_arch_back.stl" scale=" .001 .001 .001"/>
 				</geometry>
 			</collision>
@@ -176,5 +176,5 @@
 				<origin xyz="0 0 0" rpy="0 0 0"/>
 				<geometry>
-					<mesh filename="package://softfoot_thing_description/meshes/visual/roll_link_v04.stl" scale=" .001 .001 .001"/>
+                                        <mesh filename="package://softfoot_thing_description/meshes/collision/roll_link_v04.stl" scale=" .001 .001 .001"/>
 				</geometry>
 			</collision>
@@ -217,5 +217,5 @@
 				<origin xyz="0 0 0" rpy="0 0 0"/>
 				<geometry>
-					<mesh filename="package://softfoot_thing_description/meshes/visual/roll_link_v04.stl" scale=" .001 .001 .001"/>
+                                        <mesh filename="package://softfoot_thing_description/meshes/collision/roll_link_v04.stl" scale=" .001 .001 .001"/>
 				</geometry>
 			</collision>

Commit message: Changed realistic effort and velocity limits

File: softfoot_thing_description/model/chain_thing.urdf.xacro (robot description, xacro)
@@ -5,6 +5,6 @@
 	<xacro:property name="inner_chain_mass" value="0.0082"/>
 	<xacro:property name="outer_chain_mass" value="0.0156"/>
-	<xacro:property name="velocity_scale" value="1"/>
-	<xacro:property name="effort_scale" value="1"/>
+	<xacro:property name="velocity" value="100" />
+	<xacro:property name="effort" value="100" />
 	<!-- Utilities -->
     <xacro:include filename="$(find softfoot_thing_description)/model/chain_thing_inertia.xacro"/>
@@ -18,5 +18,5 @@
 			<origin xyz="0 0 0" rpy="0 0 0"/>
 			<axis xyz="1 0 0"/>
-                        <limit lower="${-45 * const_pi / 180}" upper="${45 * const_pi / 180}" effort="1" velocity="1" />
+                        <limit lower="${-45 * const_pi / 180}" upper="${45 * const_pi / 180}" effort="${effort}" velocity="${velocity}" />
 			<dynamics friction="0.0001" damping="0.0001"/>
 			<parent link="${parent}"/>
@@ -47,5 +47,5 @@
 			<origin xyz="0 0 0.0127" rpy="0 0 0"/>
 			<axis xyz="1 0 0"/>
-                        <limit lower="${-45 * const_pi / 180}" upper="${45 * const_pi / 180}" effort="1" velocity="1" />
+                        <limit lower="${-45 * const_pi / 180}" upper="${45 * const_pi / 180}" effort="${effort}" velocity="${velocity}" />
 			<dynamics friction="0.0001" damping="0.0001"/>
 			<parent link="${foot}_${name}_1_link"/>
@@ -76,5 +76,5 @@
 			<origin xyz="0 0 0.0127" rpy="0 0 0"/>
 			<axis xyz="1 0 0"/>
-                        <limit lower="${-45 * const_pi / 180}" upper="${45 * const_pi / 180}" effort="1" velocity="1" />
+                        <limit lower="${-45 * const_pi / 180}" upper="${45 * const_pi / 180}" effort="${effort}" velocity="${velocity}" />
 			<dynamics friction="0.0001" damping="0.0001"/>
 			<parent link="${foot}_${name}_2_link"/>
@@ -105,5 +105,5 @@
 			<origin xyz="0 0 0.0127" rpy="0 0 0"/>
 			<axis xyz="1 0 0"/>
-                        <limit lower="${-45 * const_pi / 180}" upper="${45 * const_pi / 180}" effort="1" velocity="1" />
+                        <limit lower="${-45 * const_pi / 180}" upper="${45 * const_pi / 180}" effort="${effort}" velocity="${velocity}" />
 			<dynamics friction="0.0001" damping="0.0001"/>
 			<parent link="${foot}_${name}_3_link"/>
@@ -134,5 +134,5 @@
 			<origin xyz="0 0 0.0127" rpy="0 0 0"/>
 			<axis xyz="1 0 0"/>
-                        <limit lower="${-45 * const_pi / 180}" upper="${45 * const_pi / 180}" effort="1" velocity="1" />
+                        <limit lower="${-45 * const_pi / 180}" upper="${45 * const_pi / 180}" effort="${effort}" velocity="${velocity}" />
 			<dynamics friction="0.0001" damping="0.0001"/>
 			<parent link="${foot}_${name}_4_link"/>
@@ -163,5 +163,5 @@
 			<origin xyz="0 0 0.0127" rpy="0 0 0"/>
 			<axis xyz="1 0 0"/>
-                        <limit lower="${-45 * const_pi / 180}" upper="${45 * const_pi / 180}" effort="1" velocity="1" />
+                        <limit lower="${-45 * const_pi / 180}" upper="${45 * const_pi / 180}" effort="${effort}" velocity="${velocity}" />
 			<dynamics friction="0.0001" damping="0.0001"/>
 			<parent link="${foot}_${name}_5_link"/>
@@ -192,5 +192,5 @@
 			<origin xyz="0 0 0.0127" rpy="0 0 0"/>
 			<axis xyz="1 0 0"/>
-                        <limit lower="${-45 * const_pi / 180}" upper="${45 * const_pi / 180}" effort="1" velocity="1" />
+                        <limit lower="${-45 * const_pi / 180}" upper="${45 * const_pi / 180}" effort="${effort}" velocity="${velocity}" />
 			<dynamics friction="0.0001" damping="0.0001"/>
 			<parent link="${foot}_${name}_6_link"/>
@@ -221,5 +221,5 @@
 			<origin xyz="0 0 0.0127" rpy="0 0 0"/>
 			<axis xyz="1 0 0"/>
-                        <limit lower="${-45 * const_pi / 180}" upper="${45 * const_pi / 180}" effort="1" velocity="1" />
+                        <limit lower="${-45 * const_pi / 180}" upper="${45 * const_pi / 180}" effort="${effort}" velocity="${velocity}" />
 			<dynamics friction="0.0001" damping="0.0001"/>
 			<parent link="${foot}_${name}_7_link"/>
@@ -250,5 +250,5 @@
 			<origin xyz="0 0 0.0127" rpy="0 0 0"/>
 			<axis xyz="1 0 0"/>
-                        <limit lower="${-45 * const_pi / 180}" upper="${45 * const_pi / 180}" effort="1" velocity="1" />
+                        <limit lower="${-45 * const_pi / 180}" upper="${45 * const_pi / 180}" effort="${effort}" velocity="${velocity}" />
 			<dynamics friction="0.0001" damping="0.0001"/>
 			<parent link="${foot}_${name}_8_link"/>
