Commit message: simplified meshes with boxes, cylinders, and spheres

File: softfoot_thing_description/model/chain_thing.urdf.xacro (robot description, xacro)
@@ -39,8 +39,7 @@
             </visual>
             <collision>
-                <origin xyz="0 0 0" rpy="0 0 0"/>
-                <geometry>
-                    <mesh filename="package://softfoot_thing_description/meshes/collision/inner_chain.stl"
-                          scale=" .001 .001 .001"/>
+                <origin xyz="0 0 0.00625" rpy="0 0 0"/>
+                <geometry>
+                    <box size="0.009 0.009 0.015"/>
                 </geometry>
             </collision>
@@ -71,8 +70,13 @@
             </visual>
             <collision>
-                <origin xyz="0 0 0" rpy="0 0 0"/>
-                <geometry>
-                    <mesh filename="package://softfoot_thing_description/meshes/collision/outer_chain.stl"
-                          scale=" .001 .001 .001"/>
+                <origin xyz="0 0.0015 0.00625" rpy="1.57079632679 0 0"/>
+                <geometry>
+                    <cylinder length="0.018" radius="0.005"/>
+                </geometry>
+            </collision>
+            <collision>
+                <origin xyz="0 0.0105 0.00625" rpy="0 0 0"/>
+                <geometry>
+                    <sphere radius="0.005"/>
                 </geometry>
             </collision>
@@ -103,8 +107,7 @@
             </visual>
             <collision>
-                <origin xyz="0 0 0" rpy="0 0 0"/>
-                <geometry>
-                    <mesh filename="package://softfoot_thing_description/meshes/collision/inner_chain.stl"
-                          scale=" .001 .001 .001"/>
+                <origin xyz="0 0 0.00625" rpy="0 0 0"/>
+                <geometry>
+                    <box size="0.009 0.009 0.015"/>
                 </geometry>
             </collision>
@@ -135,8 +138,13 @@
             </visual>
             <collision>
-                <origin xyz="0 0 0" rpy="0 0 0"/>
-                <geometry>
-                    <mesh filename="package://softfoot_thing_description/meshes/collision/outer_chain.stl"
-                          scale=" .001 .001 .001"/>
+                <origin xyz="0 0.0015 0.00625" rpy="1.57079632679 0 0"/>
+                <geometry>
+                    <cylinder length="0.018" radius="0.005"/>
+                </geometry>
+            </collision>
+            <collision>
+                <origin xyz="0 0.0105 0.00625" rpy="0 0 0"/>
+                <geometry>
+                    <sphere radius="0.005"/>
                 </geometry>
             </collision>
@@ -167,8 +175,7 @@
             </visual>
             <collision>
-                <origin xyz="0 0 0" rpy="0 0 0"/>
-                <geometry>
-                    <mesh filename="package://softfoot_thing_description/meshes/collision/inner_chain.stl"
-                          scale=" .001 .001 .001"/>
+                <origin xyz="0 0 0.00625" rpy="0 0 0"/>
+                <geometry>
+                    <box size="0.009 0.009 0.015"/>
                 </geometry>
             </collision>
@@ -199,8 +206,13 @@
             </visual>
             <collision>
-                <origin xyz="0 0 0" rpy="0 0 0"/>
-                <geometry>
-                    <mesh filename="package://softfoot_thing_description/meshes/collision/outer_chain.stl"
-                          scale=" .001 .001 .001"/>
+                <origin xyz="0 0.0015 0.00625" rpy="1.57079632679 0 0"/>
+                <geometry>
+                    <cylinder length="0.018" radius="0.005"/>
+                </geometry>
+            </collision>
+            <collision>
+                <origin xyz="0 0.0105 0.00625" rpy="0 0 0"/>
+                <geometry>
+                    <sphere radius="0.005"/>
                 </geometry>
             </collision>
@@ -231,8 +243,7 @@
             </visual>
             <collision>
-                <origin xyz="0 0 0" rpy="0 0 0"/>
-                <geometry>
-                    <mesh filename="package://softfoot_thing_description/meshes/collision/inner_chain.stl"
-                          scale=" .001 .001 .001"/>
+                <origin xyz="0 0 0.00625" rpy="0 0 0"/>
+                <geometry>
+                    <box size="0.009 0.009 0.015"/>
                 </geometry>
             </collision>
@@ -263,8 +274,13 @@
             </visual>
             <collision>
-                <origin xyz="0 0 0" rpy="0 0 0"/>
-                <geometry>
-                    <mesh filename="package://softfoot_thing_description/meshes/collision/outer_chain.stl"
-                          scale=" .001 .001 .001"/>
+                <origin xyz="0 0.0015 0.00625" rpy="1.57079632679 0 0"/>
+                <geometry>
+                    <cylinder length="0.018" radius="0.005"/>
+                </geometry>
+            </collision>
+            <collision>
+                <origin xyz="0 0.0105 0.00625" rpy="0 0 0"/>
+                <geometry>
+                    <sphere radius="0.005"/>
                 </geometry>
             </collision>
@@ -295,8 +311,7 @@
             </visual>
             <collision>
-                <origin xyz="0 0 0" rpy="0 0 0"/>
-                <geometry>
-                    <mesh filename="package://softfoot_thing_description/meshes/collision/inner_chain.stl"
-                          scale=" .001 .001 .001"/>
+                <origin xyz="0 0 0.00625" rpy="0 0 0"/>
+                <geometry>
+                    <box size="0.009 0.009 0.015"/>
                 </geometry>
             </collision>

File: softfoot_thing_description/model/softfoot_thing.urdf.xacro (robot description, xacro)
@@ -53,8 +53,25 @@
             </visual>
             <collision>
-                <origin xyz="0 0 0" rpy="0 0 0"/>
-                <geometry>
-                    <mesh filename="package://softfoot_thing_description/meshes/collision/ankle.stl"
-                          scale=" .001 .001 .001"/>
+                <origin xyz="0 0 0.02225" rpy="0 0 0"/>
+                <geometry>
+                    <cylinder length="0.0045" radius="0.02"/>
+                </geometry>
+            </collision>
+            <collision>
+                <origin xyz="0 0 0.019" rpy="0 0 0"/>
+                <geometry>
+                    <box size="0.0125 0.038 0.004"/>
+                </geometry>
+            </collision>
+            <collision>
+                <origin xyz="0 0.017 0.008" rpy="0 0 0"/>
+                <geometry>
+                    <box size="0.0125 0.004 0.028"/>
+                </geometry>
+            </collision>
+            <collision>
+                <origin xyz="0 -0.017 0.008" rpy="0 0 0"/>
+                <geometry>
+                    <box size="0.0125 0.004 0.028"/>
                 </geometry>
             </collision>
@@ -84,21 +101,28 @@
             </visual>
             <collision>
-                <origin xyz="0 0 0" rpy="0 0 0"/>
-                <geometry>
-                    <mesh filename="package://softfoot_thing_description/meshes/collision/front_arch_front.stl"
-                          scale=" .001 .001 .001"/>
-                </geometry>
-            </collision>
-        </link>
-        <!-- 2) Front arch - stiffness -->
-        <!-- <joint name="${name}_front_arch_joint_stiffness" type="revolute">
-                <origin xyz="0 0 0" rpy="0 0 0"/>
-    <axis xyz="0 1 0"/>
-    <limit lower="${min_stiffness}" upper="${max_stiffness}" effort="0" velocity="${rate_stiffness}" />
-    <safety_controller soft_lower_limit="${min_stiffness}" soft_upper_limit="${max_stiffness}" k_position="10" k_velocity="10"/>
-    <parent link="${name}_ankle_link"/>
-    <child link="${name}_front_arch_dummy"/>
-</joint>
-<link name="${name}_front_arch_dummy"/> -->
+                <origin xyz="0.01 0 0" rpy="0 0 0"/>
+                <geometry>
+                    <box size="0.03 0.029 0.008"/>
+                </geometry>
+            </collision>
+            <collision>
+                <origin xyz="0.0365 0 -0.00375" rpy="0 0.3 0"/>
+                <geometry>
+                    <box size="0.0275 0.025 0.008"/>
+                </geometry>
+            </collision>
+            <collision>
+                <origin xyz="0.05525 0 -0.0142" rpy="0 0.75 0"/>
+                <geometry>
+                    <box size="0.021 0.021 0.009"/>
+                </geometry>
+            </collision>
+            <collision>
+                <origin xyz="0.0605 0 -0.025" rpy="0 1.57 0"/>
+                <geometry>
+                    <cylinder length="0.0125" radius="0.0075"/>
+                </geometry>
+            </collision>
+        </link>
         <!-- 3) Back arch - joint along y-axis to pitch -->
         <joint name="${name}_back_arch_joint" type="revolute">
@@ -125,21 +149,28 @@
             </visual>
             <collision>
-                <origin xyz="0 0 0" rpy="0 0 0"/>
-                <geometry>
-                    <mesh filename="package://softfoot_thing_description/meshes/collision/front_arch_back.stl"
-                          scale=" .001 .001 .001"/>
-                </geometry>
-            </collision>
-        </link>
-        <!-- 3) Back arch - stiffness -->
-        <!-- <joint name="${name}_back_arch_joint_stiffness" type="revolute">
-                <origin xyz="0 0 0" rpy="0 0 0"/>
-    <axis xyz="0 -1 0"/>
-    <limit lower="${min_stiffness}" upper="${max_stiffness}" effort="0" velocity="${rate_stiffness}" />
-    <safety_controller soft_lower_limit="${min_stiffness}" soft_upper_limit="${max_stiffness}" k_position="10" k_velocity="10"/>
-    <parent link="${name}_ankle_link"/>
-    <child link="${name}_back_arch_dummy"/>
-</joint>
-<link name="${name}_back_arch_dummy"/> -->
+                <origin xyz="-0.01 0 0" rpy="0 0 0"/>
+                <geometry>
+                    <box size="0.03 0.029 0.008"/>
+                </geometry>
+            </collision>
+            <collision>
+                <origin xyz="-0.0365 0 -0.00375" rpy="0 -0.3 0"/>
+                <geometry>
+                    <box size="0.0275 0.025 0.008"/>
+                </geometry>
+            </collision>
+            <collision>
+                <origin xyz="-0.05525 0 -0.0142" rpy="0 -0.75 0"/>
+                <geometry>
+                    <box size="0.021 0.021 0.009"/>
+                </geometry>
+            </collision>
+            <collision>
+                <origin xyz="-0.0605 0 -0.025" rpy="0 -1.57 0"/>
+                <geometry>
+                    <cylinder length="0.0125" radius="0.0075"/>
+                </geometry>
+            </collision>
+        </link>
         <!-- x) Roll driving joint - we suppose the roll joints move specularly -->
         <joint name="${name}_roll_joint" type="revolute">
@@ -181,22 +212,10 @@
             </visual>
             <collision>
-                <origin xyz="0 0 0" rpy="0 0 0"/>
-                <geometry>
-                    <mesh filename="package://softfoot_thing_description/meshes/collision/roll_link_v04.stl"
-                          scale=" .001 .001 .001"/>
-                </geometry>
-            </collision>
-        </link>
-        <!-- 4) Front roll - stiffness -->
-        <!-- <joint name="${name}_front_roll_joint_stiffness" type="revolute">
-                <origin xyz="0.058 0 -0.028" rpy="0 -0.1047 0"/>
-    <axis xyz="1 0 0"/>
-    <limit lower="${min_stiffness}" upper="${max_stiffness}" effort="0" velocity="${rate_stiffness}" />
-    <mimic joint="${name}_roll_joint" multiplier="1"/>
-    <safety_controller soft_lower_limit="${min_stiffness}" soft_upper_limit="${max_stiffness}" k_position="10" k_velocity="10"/>
-    <parent link="${name}_front_arch_link"/>
-    <child link="${name}_front_roll_dummy"/>
-</joint>
-<link name="${name}_front_roll_dummy"/> -->
+                <origin xyz="0 0 -0.0125" rpy="0 0.1 0"/>
+                <geometry>
+                    <box size="0.015 0.055 0.017"/>
+                </geometry>
+            </collision>
+        </link>
         <!-- 4) Back roll - joint along x-axis to roll -->
         <joint name="${name}_back_roll_joint" type="revolute">
@@ -224,8 +243,7 @@
             </visual>
             <collision>
-                <origin xyz="0 0 0" rpy="0 0 0"/>
-                <geometry>
-                    <mesh filename="package://softfoot_thing_description/meshes/collision/roll_link_v04.stl"
-                          scale=" .001 .001 .001"/>
+                <origin xyz="0 0 -0.0125" rpy="0 0.1 0"/>
+                <geometry>
+                    <box size="0.015 0.055 0.017"/>
                 </geometry>
             </collision>
