Commit message: Minor changes but meshes seem heavy

File: softfoot_thing_description/model/softfoot_thing.gazebo.xacro (robot description, xacro)
@@ -18,21 +18,21 @@
 		<gazebo reference="${name}_ankle_link">
 			<gravity>true</gravity>
-			<material>Gazebo/Grey</material>
+			<!-- <material>Gazebo/Grey</material> -->
 		</gazebo>
 		<gazebo reference="${name}_front_arch_link">
 			<gravity>true</gravity>
-			<material>Gazebo/Grey</material>
+			<!-- <material>Gazebo/Grey</material> -->
 		</gazebo>
 		<gazebo reference="${name}_back_arch_link">
 			<gravity>true</gravity>
-			<material>Gazebo/Grey</material>
+			<!-- <material>Gazebo/Grey</material> -->
 		</gazebo>
 		<gazebo reference="${name}_front_roll_link">
 			<gravity>true</gravity>
-			<material>Gazebo/Grey</material>
+			<!-- <material>Gazebo/Grey</material> -->
 		</gazebo>
 		<gazebo reference="${name}_back_roll_link">
 			<gravity>true</gravity>
-			<material>Gazebo/Grey</material>
+			<!-- <material>Gazebo/Grey</material> -->
 		</gazebo>
 	</xacro:macro>

File: softfoot_thing_description/robot/pisa_softfoot.urdf.xacro (robot description, xacro)
@@ -8,5 +8,5 @@
   <!-- LEG -->
   <joint name="world_to_leg" type="fixed">
-    <origin xyz="0 0 0.2" rpy="0.0 0.0 0.0"/>
+    <origin xyz="0 0 0.2" rpy="0.57 0.57 0.57"/>
     <parent link="world"/>
     <child link="leg_link"/>

Commit message: Trying to debug grey model and back roll moving slowly

File: softfoot_thing_description/model/softfoot_thing.gazebo.xacro (robot description, xacro)
@@ -11,5 +11,5 @@
        		<plugin name="joint_state_publisher" filename="libgazebo_ros_joint_state_publisher.so">
          		<robotNamespace>/${name}</robotNamespace>
-         		<jointName>${name}_back_arch_joint, ${name}_front_arch_joint, ${name}_roll_joint</jointName>
+         		<jointName>${name}_front_arch_joint, ${name}_back_arch_joint, ${name}_roll_joint, ${name}_front_roll_joint, ${name}_back_roll_joint</jointName>
          		<updateRate>10.0</updateRate>
          		<alwaysOn>true</alwaysOn>

File: softfoot_thing_description/model/softfoot_thing.urdf.xacro (robot description, xacro)
@@ -155,5 +155,5 @@
 			<limit lower="${-45 * const_pi / 180}" upper="${45 * const_pi / 180}" effort="1" velocity="${velocity_scale * 45 * const_pi / 180}" />
 			<dynamics friction="0.01" damping="0.01"/>
-            <mimic joint="${name}_roll_joint" multiplier="1"/>
+            <!-- <mimic joint="${name}_roll_joint" multiplier="1"/> -->
 			<parent link="${name}_front_arch_link"/>
 			<child link="${name}_front_roll_link"/>
@@ -196,5 +196,5 @@
 			<limit lower="${-45 * const_pi / 180}" upper="${45 * const_pi / 180}" effort="1" velocity="${velocity_scale * 45 * const_pi / 180}" />
 			<dynamics friction="0.01" damping="0.01"/>
-            <mimic joint="${name}_roll_joint" multiplier="-1"/>
+            <!-- <mimic joint="${name}_roll_joint" multiplier="-1"/> -->
 			<parent link="${name}_back_arch_link"/>
 			<child link="${name}_back_roll_link"/>

Commit message: Solved some minor bugs

File: softfoot_thing_description/model/softfoot_thing.gazebo.xacro (robot description, xacro)
@@ -10,5 +10,5 @@
 		<gazebo>
        		<plugin name="joint_state_publisher" filename="libgazebo_ros_joint_state_publisher.so">
-         		<robotNamespace>/${name}</robotNamespace>
+         		<robotNamespace>${name}</robotNamespace>
          		<jointName>${name}_front_arch_joint, ${name}_back_arch_joint, ${name}_roll_joint, ${name}_front_roll_joint, ${name}_back_roll_joint</jointName>
          		<updateRate>10.0</updateRate>

File: softfoot_thing_description/model/softfoot_thing_inertia.xacro (robot description, xacro)
@@ -1,5 +1,5 @@
 <?xml version="1.0"?>
 <robot xmlns:xacro="http://www.ros.org/wiki/xacro">
-  <xacro:property name="negligible_mass" value="0.1"/>
+  <xacro:property name="negligible_mass" value="00000.1"/>
   <xacro:property name="mm2tom2" value="0.000001"/>
   <!-- INERTIA MATRICES FOR LINKS (wrt frames in urdf inertial) -->
@@ -42,5 +42,6 @@
       <origin xyz="0 0 0"/>
       <mass value="${negligible_mass}"/>
-      <inertia ixx="0.001" iyy="0.001" izz="0.001" ixy="0.0" ixz="0.0" iyz="0.0"/>
+      <inertia  ixx="${mm2tom2 * 0.0001}" iyy="${mm2tom2 * 0.0001}" izz="${mm2tom2 * 0.0001}"
+                ixy="0.0" ixz="0.0" iyz="0.0"/>
   </xacro:property>
 </robot>

File: softfoot_thing_description/robot/pisa_softfoot.urdf.xacro (robot description, xacro)
@@ -8,5 +8,5 @@
   <!-- LEG -->
   <joint name="world_to_leg" type="fixed">
-    <origin xyz="0 0 0.2" rpy="0.0 0.0 0.0"/>
+    <origin xyz="0 0 0.2" rpy="0.78 0.78 0.78"/>
     <parent link="world"/>
     <child link="leg_link"/>
@@ -18,5 +18,4 @@
       </geometry>
       <material name="material.metal">
-        <texture />
         <color rgba="0.1 0.1 0.1 1" />
       </material>

Commit message: Material enabled for gazebo

File: softfoot_thing_description/model/softfoot_thing.gazebo.xacro (robot description, xacro)
@@ -18,21 +18,21 @@
 		<gazebo reference="${name}_ankle_link">
 			<gravity>true</gravity>
-			<!-- <material>Gazebo/Grey</material> -->
+			<material>Gazebo/Grey</material>
 		</gazebo>
 		<gazebo reference="${name}_front_arch_link">
 			<gravity>true</gravity>
-			<!-- <material>Gazebo/Grey</material> -->
+			<material>Gazebo/Grey</material>
 		</gazebo>
 		<gazebo reference="${name}_back_arch_link">
 			<gravity>true</gravity>
-			<!-- <material>Gazebo/Grey</material> -->
+			<material>Gazebo/Grey</material>
 		</gazebo>
 		<gazebo reference="${name}_front_roll_link">
 			<gravity>true</gravity>
-			<!-- <material>Gazebo/Grey</material> -->
+			<material>Gazebo/Grey</material>
 		</gazebo>
 		<gazebo reference="${name}_back_roll_link">
 			<gravity>true</gravity>
-			<!-- <material>Gazebo/Grey</material> -->
+			<material>Gazebo/Grey</material>
 		</gazebo>
 	</xacro:macro>

File: softfoot_thing_description/robot/pisa_softfoot.urdf.xacro (robot description, xacro)
@@ -38,4 +38,8 @@
 		</collision>
   </link>
+  <gazebo reference="leg_link">
+			<gravity>true</gravity>
+			<material>Gazebo/Black</material>
+		</gazebo>
   <!-- FOOT -->
   <xacro:softfoot_thing name="softfoot_3" parent="leg_link">

Commit message: Indentation update

File: softfoot_thing_description/model/softfoot_thing.gazebo.xacro (robot description, xacro)
@@ -1,115 +1,105 @@
 <?xml version="1.0"?>
 <robot xmlns:xacro="http://www.ros.org/wiki/xacro">
-	<xacro:macro name="softfoot_thing_gazebo" params="name chain_name">
-		<!-- Ros control (For future actuated case) -->
-		<!-- <gazebo>
-            <plugin name="gazebo_ros_control" filename="libgazebo_ros_control.so">
+    <xacro:macro name="softfoot_thing_gazebo" params="name chain_name">
+        <!-- Ros control (For future actuated case) -->
+        <!-- <gazebo>
+                <plugin name="gazebo_ros_control" filename="libgazebo_ros_control.so">
+                    <robotNamespace>${name}</robotNamespace>
+                </plugin>
+            </gazebo> -->
+        <!-- Custom simulation plugin -->
+        <gazebo>
+                <plugin name="${name}_gazebo_sim" filename="libsoftfoot_thing_gazebo_plugin.so">
+                        <robotNamespace>${name}</robotNamespace>
+                </plugin>
+        </gazebo>
+        <!-- Provide joint feedback when simulating -->
+        <gazebo>
+        <plugin name="joint_state_publisher" filename="libgazebo_ros_joint_state_publisher.so">
                 <robotNamespace>${name}</robotNamespace>
-            </plugin>
-        </gazebo> -->
-		<!-- Custom simulation plugin -->
-		<gazebo>
-			<plugin name="${name}_gazebo_sim" filename="libsoftfoot_thing_gazebo_plugin.so">
-				<robotNamespace>${name}</robotNamespace>
-			</plugin>
-		</gazebo>
-		<!-- Provide joint feedback when simulating -->
-		<gazebo>
-       		<plugin name="joint_state_publisher" filename="libgazebo_ros_joint_state_publisher.so">
-         		<robotNamespace>${name}</robotNamespace>
-         		<jointName>	${name}_front_arch_joint, ${name}_back_arch_joint,
-                                        ${name}_roll_joint, ${name}_front_roll_joint,
-                                        ${name}_back_roll_joint, ${name}_${chain_name}_1_joint,
-                                        ${name}_${chain_name}_2_joint, ${name}_${chain_name}_3_joint,
-                                        ${name}_${chain_name}_4_joint, ${name}_${chain_name}_5_joint,
-                                        ${name}_${chain_name}_6_joint, ${name}_${chain_name}_7_joint,
-                                        ${name}_${chain_name}_8_joint, ${name}_${chain_name}_9_joint
-                        </jointName>
-         		<updateRate>10.0</updateRate>
-         		<alwaysOn>true</alwaysOn>
-       		</plugin>
-   		</gazebo>
-		<!-- Foot -->
-		<gazebo reference="${name}_ankle_link">
-			<gravity>true</gravity>
-			<!-- <selfCollide>true</selfCollide> -->
-			<material>Gazebo/Grey</material>
-		</gazebo>
-		<gazebo reference="${name}_front_arch_link">
-			<gravity>true</gravity>
-			<!-- <selfCollide>true</selfCollide> -->
-			<material>Gazebo/Grey</material>
-		</gazebo>
-		<gazebo reference="${name}_back_arch_link">
-			<gravity>true</gravity>
-			<!-- <selfCollide>true</selfCollide> -->
-			<material>Gazebo/Grey</material>
-		</gazebo>
-		<gazebo reference="${name}_front_roll_link">
-			<gravity>true</gravity>
-			<selfCollide>true</selfCollide>
-			<material>Gazebo/Grey</material>
-		</gazebo>
-		<gazebo reference="${name}_back_roll_link">
-			<gravity>true</gravity>
-			<selfCollide>true</selfCollide>
-			<material>Gazebo/Grey</material>
-		</gazebo>
-                <gazebo reference="${name}_${chain_name}_insertion_link">
-                        <gravity>true</gravity>
-                        <!--<selfCollide>true</selfCollide>-->
-                        <material>Gazebo/Grey</material>
-                </gazebo>
-		<!-- Chain -->
-		<gazebo reference="${name}_${chain_name}_1_link">
-			<gravity>true</gravity>
-			<!-- <selfCollide>true</selfCollide> -->
-			<material>Gazebo/Grey</material>
-		</gazebo>
-		<gazebo reference="${name}_${chain_name}_2_link">
-			<gravity>true</gravity>
-			<!-- <selfCollide>true</selfCollide> -->
-			<material>Gazebo/Grey</material>
-		</gazebo>
-		<gazebo reference="${name}_${chain_name}_3_link">
-			<gravity>true</gravity>
-			<!-- <selfCollide>true</selfCollide> -->
-			<material>Gazebo/Grey</material>
-		</gazebo>
-		<gazebo reference="${name}_${chain_name}_4_link">
-			<gravity>true</gravity>
-			<!-- <selfCollide>true</selfCollide> -->
-			<material>Gazebo/Grey</material>
-		</gazebo>
-		<gazebo reference="${name}_${chain_name}_5_link">
-			<gravity>true</gravity>
-			<!-- <selfCollide>true</selfCollide> -->
-			<material>Gazebo/Grey</material>
-		</gazebo>
-		<gazebo reference="${name}_${chain_name}_6_link">
-			<gravity>true</gravity>
-			<!-- <selfCollide>true</selfCollide> -->
-			<material>Gazebo/Grey</material>
-		</gazebo>
-		<gazebo reference="${name}_${chain_name}_7_link">
-			<gravity>true</gravity>
-			<!-- <selfCollide>true</selfCollide> -->
-			<material>Gazebo/Grey</material>
-		</gazebo>
-		<gazebo reference="${name}_${chain_name}_8_link">
-			<gravity>true</gravity>
-			<!-- <selfCollide>true</selfCollide> -->
-			<material>Gazebo/Grey</material>
-		</gazebo>
-		<gazebo reference="${name}_${chain_name}_9_link">
-			<gravity>true</gravity>
-			<!-- <selfCollide>true</selfCollide> -->
-			<material>Gazebo/Grey</material>
-		</gazebo>
-                <gazebo reference="${name}_${chain_name}_tip_link">
-                        <gravity>true</gravity>
-                        <!-- <selfCollide>true</selfCollide> -->
-                        <material>Gazebo/Grey</material>
-                </gazebo>
-	</xacro:macro>
+                <jointName>	${name}_front_arch_joint, ${name}_back_arch_joint,
+                                ${name}_roll_joint, ${name}_front_roll_joint,
+                                ${name}_back_roll_joint, ${name}_${chain_name}_1_joint,
+                                ${name}_${chain_name}_2_joint, ${name}_${chain_name}_3_joint,
+                                ${name}_${chain_name}_4_joint, ${name}_${chain_name}_5_joint,
+                                ${name}_${chain_name}_6_joint, ${name}_${chain_name}_7_joint,
+                                ${name}_${chain_name}_8_joint, ${name}_${chain_name}_9_joint
+                </jointName>
+                <updateRate>10.0</updateRate>
+                <alwaysOn>true</alwaysOn>
+        </plugin>
+        </gazebo>
+        <!-- Foot -->
+        <gazebo reference="${name}_ankle_link">
+                <gravity>true</gravity>
+                <!-- <selfCollide>true</selfCollide> -->
+                <material>Gazebo/Grey</material>
+        </gazebo>
+        <gazebo reference="${name}_front_arch_link">
+                <gravity>true</gravity>
+                <!-- <selfCollide>true</selfCollide> -->
+                <material>Gazebo/Grey</material>
+        </gazebo>
+        <gazebo reference="${name}_back_arch_link">
+                <gravity>true</gravity>
+                <!-- <selfCollide>true</selfCollide> -->
+                <material>Gazebo/Grey</material>
+        </gazebo>
+        <gazebo reference="${name}_front_roll_link">
+                <gravity>true</gravity>
+                <selfCollide>true</selfCollide>
+                <material>Gazebo/Grey</material>
+        </gazebo>
+        <gazebo reference="${name}_back_roll_link">
+                <gravity>true</gravity>
+                <selfCollide>true</selfCollide>
+                <material>Gazebo/Grey</material>
+        </gazebo>
+        <!-- Chain -->
+        <gazebo reference="${name}_${chain_name}_1_link">
+                <gravity>true</gravity>
+                <!-- <selfCollide>true</selfCollide> -->
+                <material>Gazebo/Grey</material>
+        </gazebo>
+        <gazebo reference="${name}_${chain_name}_2_link">
+                <gravity>true</gravity>
+                <!-- <selfCollide>true</selfCollide> -->
+                <material>Gazebo/Grey</material>
+        </gazebo>
+        <gazebo reference="${name}_${chain_name}_3_link">
+                <gravity>true</gravity>
+                <!-- <selfCollide>true</selfCollide> -->
+                <material>Gazebo/Grey</material>
+        </gazebo>
+        <gazebo reference="${name}_${chain_name}_4_link">
+                <gravity>true</gravity>
+                <!-- <selfCollide>true</selfCollide> -->
+                <material>Gazebo/Grey</material>
+        </gazebo>
+        <gazebo reference="${name}_${chain_name}_5_link">
+                <gravity>true</gravity>
+                <!-- <selfCollide>true</selfCollide> -->
+                <material>Gazebo/Grey</material>
+        </gazebo>
+        <gazebo reference="${name}_${chain_name}_6_link">
+                <gravity>true</gravity>
+                <!-- <selfCollide>true</selfCollide> -->
+                <material>Gazebo/Grey</material>
+        </gazebo>
+        <gazebo reference="${name}_${chain_name}_7_link">
+                <gravity>true</gravity>
+                <!-- <selfCollide>true</selfCollide> -->
+                <material>Gazebo/Grey</material>
+        </gazebo>
+        <gazebo reference="${name}_${chain_name}_8_link">
+                <gravity>true</gravity>
+                <!-- <selfCollide>true</selfCollide> -->
+                <material>Gazebo/Grey</material>
+        </gazebo>
+        <gazebo reference="${name}_${chain_name}_9_link">
+                <gravity>true</gravity>
+                <!-- <selfCollide>true</selfCollide> -->
+                <material>Gazebo/Grey</material>
+        </gazebo>
+    </xacro:macro>
 </robot>
