Commit message: Improved contact parameters

File: softfoot_thing_description/model/softfoot_thing.gazebo.xacro (robot description, xacro)
@@ -1,22 +1,22 @@
 <?xml version="1.0"?>
 <robot xmlns:xacro="http://www.ros.org/wiki/xacro">
-    <xacro:macro name="softfoot_thing_gazebo" params="name left_chain_name middle_chain_name right_chain_name">
-        <!-- Ros control (For future actuated case) -->
-        <!-- <gazebo>
+        <xacro:macro name="softfoot_thing_gazebo" params="name left_chain_name middle_chain_name right_chain_name">
+                <!-- Ros control (For future actuated case) -->
+                <!-- <gazebo>
                 <plugin name="gazebo_ros_control" filename="libgazebo_ros_control.so">
                     <robotNamespace>${name}</robotNamespace>
                 </plugin>
             </gazebo> -->
-        <!-- Custom simulation plugin -->
-        <gazebo>
-                <plugin name="${name}_gazebo_sim" filename="libsoftfoot_thing_gazebo_plugin.so">
-                        <robotNamespace>${name}</robotNamespace>
-                </plugin>
-        </gazebo>
-        <!-- Provide joint feedback when simulating -->
-        <gazebo>
-        <plugin name="joint_state_publisher" filename="libgazebo_ros_joint_state_publisher.so">
-                <robotNamespace>${name}</robotNamespace>
-                <jointName>	${name}_front_arch_joint, ${name}_back_arch_joint,
+                <!-- Custom simulation plugin -->
+                <gazebo>
+                        <plugin name="${name}_gazebo_sim" filename="libsoftfoot_thing_gazebo_plugin.so">
+                                <robotNamespace>${name}</robotNamespace>
+                        </plugin>
+                </gazebo>
+                <!-- Provide joint feedback when simulating -->
+                <gazebo>
+                        <plugin name="joint_state_publisher" filename="libgazebo_ros_joint_state_publisher.so">
+                                <robotNamespace>${name}</robotNamespace>
+                                <jointName>	${name}_front_arch_joint, ${name}_back_arch_joint,
                                 ${name}_roll_joint, ${name}_front_roll_joint,
                                 ${name}_back_roll_joint, ${name}_${left_chain_name}_1_joint,
@@ -36,172 +36,620 @@
                                 ${name}_${right_chain_name}_8_joint, ${name}_${right_chain_name}_9_joint
                 </jointName>
-                <updateRate>100.0</updateRate>
-                <alwaysOn>true</alwaysOn>
-        </plugin>
-        </gazebo>
-        <!-- Foot -->
-        <gazebo reference="${name}_ankle_link">
-                <gravity>true</gravity>
-                <!-- <selfCollide>true</selfCollide> -->
-                <material>Gazebo/Grey</material>
-        </gazebo>
-        <gazebo reference="${name}_front_arch_link">
-                <gravity>true</gravity>
-                <!-- <selfCollide>true</selfCollide> -->
-                <material>Gazebo/Grey</material>
-        </gazebo>
-        <gazebo reference="${name}_back_arch_link">
-                <gravity>true</gravity>
-                <!-- <selfCollide>true</selfCollide> -->
-                <material>Gazebo/Grey</material>
-        </gazebo>
-        <gazebo reference="${name}_front_roll_link">
-                <gravity>true</gravity>
-                <selfCollide>true</selfCollide>
-                <material>Gazebo/Grey</material>
-        </gazebo>
-        <gazebo reference="${name}_back_roll_link">
-                <gravity>true</gravity>
-                <selfCollide>true</selfCollide>
-                <material>Gazebo/Grey</material>
-        </gazebo>
-        <!-- Left Chain -->
-        <gazebo reference="${name}_${left_chain_name}_1_link">
-                <gravity>true</gravity>
-                <!-- <selfCollide>true</selfCollide> -->
-                <material>Gazebo/Grey</material>
-        </gazebo>
-        <gazebo reference="${name}_${left_chain_name}_2_link">
-                <gravity>true</gravity>
-                <!-- <selfCollide>true</selfCollide> -->
-                <material>Gazebo/Grey</material>
-        </gazebo>
-        <gazebo reference="${name}_${left_chain_name}_3_link">
-                <gravity>true</gravity>
-                <!-- <selfCollide>true</selfCollide> -->
-                <material>Gazebo/Grey</material>
-        </gazebo>
-        <gazebo reference="${name}_${left_chain_name}_4_link">
-                <gravity>true</gravity>
-                <!-- <selfCollide>true</selfCollide> -->
-                <material>Gazebo/Grey</material>
-        </gazebo>
-        <gazebo reference="${name}_${left_chain_name}_5_link">
-                <gravity>true</gravity>
-                <!-- <selfCollide>true</selfCollide> -->
-                <material>Gazebo/Grey</material>
-        </gazebo>
-        <gazebo reference="${name}_${left_chain_name}_6_link">
-                <gravity>true</gravity>
-                <!-- <selfCollide>true</selfCollide> -->
-                <material>Gazebo/Grey</material>
-        </gazebo>
-        <gazebo reference="${name}_${left_chain_name}_7_link">
-                <gravity>true</gravity>
-                <!-- <selfCollide>true</selfCollide> -->
-                <material>Gazebo/Grey</material>
-        </gazebo>
-        <gazebo reference="${name}_${left_chain_name}_8_link">
-                <gravity>true</gravity>
-                <!-- <selfCollide>true</selfCollide> -->
-                <material>Gazebo/Grey</material>
-        </gazebo>
-        <gazebo reference="${name}_${left_chain_name}_9_link">
-                <gravity>true</gravity>
-                <selfCollide>true</selfCollide>
-                <material>Gazebo/Grey</material>
-        </gazebo>
-        <!-- Middle Chain -->
-        <gazebo reference="${name}_${middle_chain_name}_1_link">
-                <gravity>true</gravity>
-                <!-- <selfCollide>true</selfCollide> -->
-                <material>Gazebo/Grey</material>
-        </gazebo>
-        <gazebo reference="${name}_${middle_chain_name}_2_link">
-                <gravity>true</gravity>
-                <!-- <selfCollide>true</selfCollide> -->
-                <material>Gazebo/Grey</material>
-        </gazebo>
-        <gazebo reference="${name}_${middle_chain_name}_3_link">
-                <gravity>true</gravity>
-                <!-- <selfCollide>true</selfCollide> -->
-                <material>Gazebo/Grey</material>
-        </gazebo>
-        <gazebo reference="${name}_${middle_chain_name}_4_link">
-                <gravity>true</gravity>
-                <!-- <selfCollide>true</selfCollide> -->
-                <material>Gazebo/Grey</material>
-        </gazebo>
-        <gazebo reference="${name}_${middle_chain_name}_5_link">
-                <gravity>true</gravity>
-                <!-- <selfCollide>true</selfCollide> -->
-                <material>Gazebo/Grey</material>
-        </gazebo>
-        <gazebo reference="${name}_${middle_chain_name}_6_link">
-                <gravity>true</gravity>
-                <!-- <selfCollide>true</selfCollide> -->
-                <material>Gazebo/Grey</material>
-        </gazebo>
-        <gazebo reference="${name}_${middle_chain_name}_7_link">
-                <gravity>true</gravity>
-                <!-- <selfCollide>true</selfCollide> -->
-                <material>Gazebo/Grey</material>
-        </gazebo>
-        <gazebo reference="${name}_${middle_chain_name}_8_link">
-                <gravity>true</gravity>
-                <!-- <selfCollide>true</selfCollide> -->
-                <material>Gazebo/Grey</material>
-        </gazebo>
-        <gazebo reference="${name}_${middle_chain_name}_9_link">
-                <gravity>true</gravity>
-                <selfCollide>true</selfCollide>
-                <material>Gazebo/Grey</material>
-        </gazebo>
-        <!-- Right Chain -->
-        <gazebo reference="${name}_${right_chain_name}_1_link">
-                <gravity>true</gravity>
-                <!-- <selfCollide>true</selfCollide> -->
-                <material>Gazebo/Grey</material>
-        </gazebo>
-        <gazebo reference="${name}_${right_chain_name}_2_link">
-                <gravity>true</gravity>
-                <!-- <selfCollide>true</selfCollide> -->
-                <material>Gazebo/Grey</material>
-        </gazebo>
-        <gazebo reference="${name}_${right_chain_name}_3_link">
-                <gravity>true</gravity>
-                <!-- <selfCollide>true</selfCollide> -->
-                <material>Gazebo/Grey</material>
-        </gazebo>
-        <gazebo reference="${name}_${right_chain_name}_4_link">
-                <gravity>true</gravity>
-                <!-- <selfCollide>true</selfCollide> -->
-                <material>Gazebo/Grey</material>
-        </gazebo>
-        <gazebo reference="${name}_${right_chain_name}_5_link">
-                <gravity>true</gravity>
-                <!-- <selfCollide>true</selfCollide> -->
-                <material>Gazebo/Grey</material>
-        </gazebo>
-        <gazebo reference="${name}_${right_chain_name}_6_link">
-                <gravity>true</gravity>
-                <!-- <selfCollide>true</selfCollide> -->
-                <material>Gazebo/Grey</material>
-        </gazebo>
-        <gazebo reference="${name}_${right_chain_name}_7_link">
-                <gravity>true</gravity>
-                <!-- <selfCollide>true</selfCollide> -->
-                <material>Gazebo/Grey</material>
-        </gazebo>
-        <gazebo reference="${name}_${right_chain_name}_8_link">
-                <gravity>true</gravity>
-                <!-- <selfCollide>true</selfCollide> -->
-                <material>Gazebo/Grey</material>
-        </gazebo>
-        <gazebo reference="${name}_${right_chain_name}_9_link">
-                <gravity>true</gravity>
-                <selfCollide>true</selfCollide>
-                <material>Gazebo/Grey</material>
-        </gazebo>
-    </xacro:macro>
+                                <updateRate>100.0</updateRate>
+                                <alwaysOn>true</alwaysOn>
+                        </plugin>
+                </gazebo>
+                <!-- Foot -->
+                <gazebo reference="${name}_ankle_link">
+                        <gravity>true</gravity>
+                        <!-- <selfCollide>true</selfCollide> -->
+                        <material>Gazebo/Grey</material>
+                        <kp>1e15</kp>
+                        <kd>1e13</kd>
+                        <mu1>0.8</mu1>
+                        <mu2>0.8</mu2>
+                        <collision>
+                                <surface>
+                                        <contact>
+                                                <ode>
+                                                        <min_depth>0.01</min_depth>
+                                                        <max_vel>0.1</max_vel>
+                                                </ode>
+                                        </contact>
+                                </surface>
+                        </collision>
+                </gazebo>
+                <gazebo reference="${name}_front_arch_link">
+                        <gravity>true</gravity>
+                        <!-- <selfCollide>true</selfCollide> -->
+                        <material>Gazebo/Grey</material>
+                        <kp>1e15</kp>
+                        <kd>1e13</kd>
+                        <mu1>0.8</mu1>
+                        <mu2>0.8</mu2>
+                        <collision>
+                                <surface>
+                                        <contact>
+                                                <ode>
+                                                        <min_depth>0.01</min_depth>
+                                                        <max_vel>0.1</max_vel>
+                                                </ode>
+                                        </contact>
+                                </surface>
+                        </collision>
+                </gazebo>
+                <gazebo reference="${name}_back_arch_link">
+                        <gravity>true</gravity>
+                        <!-- <selfCollide>true</selfCollide> -->
+                        <material>Gazebo/Grey</material>
+                        <kp>1e15</kp>
+                        <kd>1e13</kd>
+                        <mu1>0.8</mu1>
+                        <mu2>0.8</mu2>
+                        <collision>
+                                <surface>
+                                        <contact>
+                                                <ode>
+                                                        <min_depth>0.01</min_depth>
+                                                        <max_vel>0.1</max_vel>
+                                                </ode>
+                                        </contact>
+                                </surface>
+                        </collision>
+                </gazebo>
+                <gazebo reference="${name}_front_roll_link">
+                        <gravity>true</gravity>
+                        <!-- <selfCollide>true</selfCollide> -->
+                        <material>Gazebo/Grey</material>
+                        <kp>1e15</kp>
+                        <kd>1e13</kd>
+                        <mu1>0.8</mu1>
+                        <mu2>0.8</mu2>
+                        <collision>
+                                <surface>
+                                        <contact>
+                                                <ode>
+                                                        <min_depth>0.01</min_depth>
+                                                        <max_vel>0.1</max_vel>
+                                                </ode>
+                                        </contact>
+                                </surface>
+                        </collision>
+                </gazebo>
+                <gazebo reference="${name}_back_roll_link">
+                        <gravity>true</gravity>
+                        <!-- <selfCollide>true</selfCollide> -->
+                        <material>Gazebo/Grey</material>
+                        <kp>1e15</kp>
+                        <kd>1e13</kd>
+                        <mu1>0.8</mu1>
+                        <mu2>0.8</mu2>
+                        <collision>
+                                <surface>
+                                        <contact>
+                                                <ode>
+                                                        <min_depth>0.01</min_depth>
+                                                        <max_vel>0.1</max_vel>
+                                                </ode>
+                                        </contact>
+                                </surface>
+                        </collision>
+                </gazebo>
+                <!-- Left Chain -->
+                <gazebo reference="${name}_${left_chain_name}_1_link">
+                        <gravity>true</gravity>
+                        <!-- <selfCollide>true</selfCollide> -->
+                        <material>Gazebo/Grey</material>
+                        <kp>1e15</kp>
+                        <kd>1e13</kd>
+                        <mu1>0.8</mu1>
+                        <mu2>0.8</mu2>
+                        <collision>
+                                <surface>
+                                        <contact>
+                                                <ode>
+                                                        <min_depth>0.01</min_depth>
+                                                        <max_vel>0.1</max_vel>
+                                                </ode>
+                                        </contact>
+                                </surface>
+                        </collision>
+                </gazebo>
+                <gazebo reference="${name}_${left_chain_name}_2_link">
+                        <gravity>true</gravity>
+                        <!-- <selfCollide>true</selfCollide> -->
+                        <material>Gazebo/Grey</material>
+                        <kp>1e15</kp>
+                        <kd>1e13</kd>
+                        <mu1>0.8</mu1>
+                        <mu2>0.8</mu2>
+                        <collision>
+                                <surface>
+                                        <contact>
+                                                <ode>
+                                                        <min_depth>0.01</min_depth>
+                                                        <max_vel>0.1</max_vel>
+                                                </ode>
+                                        </contact>
+                                </surface>
+                        </collision>
+                </gazebo>
+                <gazebo reference="${name}_${left_chain_name}_3_link">
+                        <gravity>true</gravity>
+                        <!-- <selfCollide>true</selfCollide> -->
+                        <material>Gazebo/Grey</material>
+                        <kp>1e15</kp>
+                        <kd>1e13</kd>
+                        <mu1>0.8</mu1>
+                        <mu2>0.8</mu2>
+                        <collision>
+                                <surface>
+                                        <contact>
+                                                <ode>
+                                                        <min_depth>0.01</min_depth>
+                                                        <max_vel>0.1</max_vel>
+                                                </ode>
+                                        </contact>
+                                </surface>
+                        </collision>
+                </gazebo>
+                <gazebo reference="${name}_${left_chain_name}_4_link">
+                        <gravity>true</gravity>
+                        <!-- <selfCollide>true</selfCollide> -->
+                        <material>Gazebo/Grey</material>
+                        <kp>1e15</kp>
+                        <kd>1e13</kd>
+                        <mu1>0.8</mu1>
+                        <mu2>0.8</mu2>
+                        <collision>
+                                <surface>
+                                        <contact>
+                                                <ode>
+                                                        <min_depth>0.01</min_depth>
+                                                        <max_vel>0.1</max_vel>
+                                                </ode>
+                                        </contact>
+                                </surface>
+                        </collision>
+                </gazebo>
+                <gazebo reference="${name}_${left_chain_name}_5_link">
+                        <gravity>true</gravity>
+                        <!-- <selfCollide>true</selfCollide> -->
+                        <material>Gazebo/Grey</material>
+                        <kp>1e15</kp>
+                        <kd>1e13</kd>
+                        <mu1>0.8</mu1>
+                        <mu2>0.8</mu2>
+                        <collision>
+                                <surface>
+                                        <contact>
+                                                <ode>
+                                                        <min_depth>0.01</min_depth>
+                                                        <max_vel>0.1</max_vel>
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